File: preamp-layout/preamp-kicad/volume_encoder.sch (KiCad schematic (older format))
At the start: 0 parts

Commit message: general layout work
Changed lines of the file:
@@
 $Descr A4 11693 8268
 encoding utf-8
-Sheet 5 13
+Sheet 12 13
 Title ""
 Date ""
@@
 Comment4 ""
 $EndDescr
-Text HLabel 3600 3350 0    50   UnSpc ~ 0
-in_R
-Text HLabel 3600 3200 0    50   UnSpc ~ 0
-in_L
+Text HLabel 5150 3150 2    50   Output ~ 0
+CLK
+Text HLabel 5150 3350 2    50   Output ~ 0
+DT
+Text HLabel 5150 3550 2    50   Output ~ 0
+SW
+Text HLabel 5150 2950 2    50   Input ~ 0
+LED_DT
 $EndSCHEMATC
