File: preamp-layout/preamp-kicad/tone_control.sch (KiCad schematic (older format))
At the start: 0 parts

Commit message: readme references update. preamp-code updated to implement interrupts for encoder input. Layout general updates
Changed lines of the file:
@@
 $Descr A4 11693 8268
 encoding utf-8
-Sheet 5 11
+Sheet 10 11
 Title ""
 Date ""
@@
 Comment4 ""
 $EndDescr
-Text HLabel 3600 3350 0    50   UnSpc ~ 0
+Text HLabel 2250 4350 0    50   UnSpc ~ 0
 in_R
-Text HLabel 3600 3200 0    50   UnSpc ~ 0
+Text HLabel 2250 4200 0    50   UnSpc ~ 0
 in_L
+Text HLabel 8550 3750 2    50   UnSpc ~ 0
+out_L
+Text HLabel 8550 3900 2    50   UnSpc ~ 0
+out_R
 $EndSCHEMATC

Commit message: general layout work
Parts:
- added D? (x2): LED, symbol Device:LED
- added J? (x2): Conn_01x03_Female, symbol Connector:Conn_01x03_Female
- added J? (x2): Conn_01x03_Male, symbol Connector:Conn_01x03_Male
- added R? (x2): 10K, symbol Device:R
Connections:
- net in_L: now also J?.1 (Pin_1)
- net in_R: now also J?.2 (Pin_2)
- net out_L: now also J?.1 (Pin_1)
- net out_R: now also J?.2 (Pin_2)
- new net: D?.2 (A), R?.2
- new net: D?.1 (K), R?.2
- new net +15V: J?.1 (Pin_1), J?.1 (Pin_1), R?.1
- new net -15V: J?.2 (Pin_2), J?.2 (Pin_2), R?.1
- new net GNDA: D?.1 (K), D?.2 (A), J?.3 (Pin_3), J?.3 (Pin_3)
- new net GNDS: J?.3 (Pin_3), J?.3 (Pin_3)
Other:
- note added: "PWR, monitoring"
- note added: "Receives from IO"
- note added: "Sends to amp"
