File: preamp-layout/preamp-kicad/IO.sch (KiCad schematic (older format))
At the start: 14 parts, among them J32 Conn_Coaxial_x2, J33 Conn_Coaxial_x2, J34 Conn_Coaxial_x2, J35 Conn_Coaxial_x2, J36 Conn_Coaxial_x2, J37 Conn_01x03_Female, J38 Conn_01x03_Female, J39 Conn_01x03_Female, J40 Conn_01x03_Female, J41 Conn_01x03_Female, J42 Conn_01x03_Male, J43 Conn_01x03_Male, J44 Conn_Coaxial_x2, J45 Conn_Coaxial_x2

Commit message: AC PCB Update
Removed Switch symbol from PCB, moved to main sheet. Started playing with footprint assignment. Other minor updates.
Parts:
- renumbered J32 to J37, J33 to J38, J34 to J39, J35 to J40, J36 to J41, J37 to J42, J38 to J43, J39 to J44, J40 to J45, J41 to J46, J42 to J47, J43 to J48, J44 to J49, J45 to J50
Changed lines of the file:
@@
 P 4100 2850
 AR Path="/5E2D8DA2/5E60DD2B" Ref="J?"  Part="1"
-AR Path="/5E607732/5E60DD2B" Ref="J33"  Part="1"
-F 0 "J33" H 4028 3188 50  0000 C CNN
+AR Path="/5E607732/5E60DD2B" Ref="J38"  Part="1"
+F 0 "J38" H 4028 3188 50  0000 C CNN
 F 1 "Conn_Coaxial_x2" H 4028 3097 50  0001 C CNN
 F 2 "" H 4100 2750 50  0001 C CNN
@@
 $EndComp
 $Comp
-L Connector:Conn_01x03_Female J38
+L Connector:Conn_01x03_Female J43
 U 1 1 5E60DD36
 P 4850 2850
-F 0 "J38" H 4878 2876 50  0000 L CNN
+F 0 "J43" H 4878 2876 50  0000 L CNN
 F 1 "Conn_01x03_Female" H 4878 2785 50  0001 L CNN
 F 2 "" H 4850 2850 50  0001 C CNN
@@
 P 4100 1800
 AR Path="/5E2D8DA2/6431D3FD" Ref="J?"  Part="1"
-AR Path="/5E607732/6431D3FD" Ref="J32"  Part="1"
-F 0 "J32" H 4028 2138 50  0000 C CNN
+AR Path="/5E607732/6431D3FD" Ref="J37"  Part="1"
+F 0 "J37" H 4028 2138 50  0000 C CNN
 F 1 "Conn_Coaxial_x2" H 4028 2047 50  0001 C CNN
 F 2 "" H 4100 1700 50  0001 C CNN
@@
 $EndComp
 $Comp
-L Connector:Conn_01x03_Female J37
+L Connector:Conn_01x03_Female J42
 U 1 1 6431D407
 P 4850 1800
-F 0 "J37" H 4878 1826 50  0000 L CNN
+F 0 "J42" H 4878 1826 50  0000 L CNN
 F 1 "Conn_01x03_Female" H 4878 1735 50  0001 L CNN
 F 2 "" H 4850 1800 50  0001 C CNN
@@
 P 4100 4950
 AR Path="/5E2D8DA2/6433171F" Ref="J?"  Part="1"
-AR Path="/5E607732/6433171F" Ref="J35"  Part="1"
-F 0 "J35" H 4028 5288 50  0000 C CNN
+AR Path="/5E607732/6433171F" Ref="J40"  Part="1"
+F 0 "J40" H 4028 5288 50  0000 C CNN
 F 1 "Conn_Coaxial_x2" H 4028 5197 50  0001 C CNN
 F 2 "" H 4100 4850 50  0001 C CNN
@@
 $EndComp
 $Comp
-L Connector:Conn_01x03_Female J40
+L Connector:Conn_01x03_Female J45
 U 1 1 64331729
 P 4850 4950
-F 0 "J40" H 4878 4976 50  0000 L CNN
+F 0 "J45" H 4878 4976 50  0000 L CNN
 F 1 "Conn_01x03_Female" H 4878 4885 50  0001 L CNN
 F 2 "" H 4850 4950 50  0001 C CNN
@@
 P 4100 3900
 AR Path="/5E2D8DA2/64331754" Ref="J?"  Part="1"
-AR Path="/5E607732/64331754" Ref="J34"  Part="1"
-F 0 "J34" H 4028 4238 50  0000 C CNN
+AR Path="/5E607732/64331754" Ref="J39"  Part="1"
+F 0 "J39" H 4028 4238 50  0000 C CNN
 F 1 "Conn_Coaxial_x2" H 4028 4147 50  0001 C CNN
 F 2 "" H 4100 3800 50  0001 C CNN
@@
 $EndComp
 $Comp
-L Connector:Conn_01x03_Female J39
+L Connector:Conn_01x03_Female J44
 U 1 1 6433175E
 P 4850 3900
-F 0 "J39" H 4878 3926 50  0000 L CNN
+F 0 "J44" H 4878 3926 50  0000 L CNN
 F 1 "Conn_01x03_Female" H 4878 3835 50  0001 L CNN
 F 2 "" H 4850 3900 50  0001 C CNN
@@
 P 4100 6050
 AR Path="/5E2D8DA2/6433C001" Ref="J?"  Part="1"
-AR Path="/5E607732/6433C001" Ref="J36"  Part="1"
-F 0 "J36" H 4028 6388 50  0000 C CNN
+AR Path="/5E607732/6433C001" Ref="J41"  Part="1"
+F 0 "J41" H 4028 6388 50  0000 C CNN
 F 1 "Conn_Coaxial_x2" H 4028 6297 50  0001 C CNN
 F 2 "" H 4100 5950 50  0001 C CNN
@@
 $EndComp
 $Comp
-L Connector:Conn_01x03_Female J41
+L Connector:Conn_01x03_Female J46
 U 1 1 6433C00B
 P 4850 6050
-F 0 "J41" H 4878 6076 50  0000 L CNN
+F 0 "J46" H 4878 6076 50  0000 L CNN
 F 1 "Conn_01x03_Female" H 4878 5985 50  0001 L CNN
 F 2 "" H 4850 6050 50  0001 C CNN
@@
 P 7750 4300
 AR Path="/5E2D8DA2/64358093" Ref="J?"  Part="1"
-AR Path="/5E607732/64358093" Ref="J45"  Part="1"
-F 0 "J45" H 7678 4638 50  0000 C CNN
+AR Path="/5E607732/64358093" Ref="J50"  Part="1"
+F 0 "J50" H 7678 4638 50  0000 C CNN
 F 1 "Conn_Coaxial_x2" H 7678 4547 50  0001 C CNN
 F 2 "" H 7750 4200 50  0001 C CNN
@@
 P 7750 3250
 AR Path="/5E2D8DA2/64354C54" Ref="J?"  Part="1"
-AR Path="/5E607732/64354C54" Ref="J44"  Part="1"
-F 0 "J44" H 7678 3588 50  0000 C CNN
+AR Path="/5E607732/64354C54" Ref="J49"  Part="1"
+F 0 "J49" H 7678 3588 50  0000 C CNN
 F 1 "Conn_Coaxial_x2" H 7678 3497 50  0001 C CNN
 F 2 "" H 7750 3150 50  0001 C CNN
@@
 $EndComp
 $Comp
-L Connector:Conn_01x03_Male J42
+L Connector:Conn_01x03_Male J47
 U 1 1 6436D21D
 P 7000 3250
-F 0 "J42" H 6972 3228 50  0000 R CNN
+F 0 "J47" H 6972 3228 50  0000 R CNN
 F 1 "Conn_01x03_Male" H 6972 3183 50  0001 R CNN
 F 2 "" H 7000 3250 50  0001 C CNN
@@
 $EndComp
 $Comp
-L Connector:Conn_01x03_Male J43
+L Connector:Conn_01x03_Male J48
 U 1 1 6437A2AD
 P 7000 4300
-F 0 "J43" H 6972 4278 50  0000 R CNN
+F 0 "J48" H 6972 4278 50  0000 R CNN
 F 1 "Conn_01x03_Male" H 6972 4233 50  0001 R CNN
 F 2 "" H 7000 4300 50  0001 C CNN

Commit message: Initial Footprint Assignment
Assigned footprints to SMT resistors, pin headers, screw terminals, LEDs, DIP-8 ICs
Parts:
- J42, J43, J44, J45, J46, J47, J48: footprint (none) -> Connector_PinHeader_2.54mm:PinHeader_1x03_P2.54mm_Vertical
Changed lines of the file:
@@
 F 0 "J43" H 4878 2876 50  0000 L CNN
 F 1 "Conn_01x03_Female" H 4878 2785 50  0001 L CNN
-F 2 "" H 4850 2850 50  0001 C CNN
+F 2 "Connector_PinHeader_2.54mm:PinHeader_1x03_P2.54mm_Vertical" H 4850 2850 50  0001 C CNN
 F 3 "~" H 4850 2850 50  0001 C CNN
 	1    4850 2850
@@
 F 0 "J42" H 4878 1826 50  0000 L CNN
 F 1 "Conn_01x03_Female" H 4878 1735 50  0001 L CNN
-F 2 "" H 4850 1800 50  0001 C CNN
+F 2 "Connector_PinHeader_2.54mm:PinHeader_1x03_P2.54mm_Vertical" H 4850 1800 50  0001 C CNN
 F 3 "~" H 4850 1800 50  0001 C CNN
 	1    4850 1800
@@
 F 0 "J45" H 4878 4976 50  0000 L CNN
 F 1 "Conn_01x03_Female" H 4878 4885 50  0001 L CNN
-F 2 "" H 4850 4950 50  0001 C CNN
+F 2 "Connector_PinHeader_2.54mm:PinHeader_1x03_P2.54mm_Vertical" H 4850 4950 50  0001 C CNN
 F 3 "~" H 4850 4950 50  0001 C CNN
 	1    4850 4950
@@
 F 0 "J44" H 4878 3926 50  0000 L CNN
 F 1 "Conn_01x03_Female" H 4878 3835 50  0001 L CNN
-F 2 "" H 4850 3900 50  0001 C CNN
+F 2 "Connector_PinHeader_2.54mm:PinHeader_1x03_P2.54mm_Vertical" H 4850 3900 50  0001 C CNN
 F 3 "~" H 4850 3900 50  0001 C CNN
 	1    4850 3900
@@
 F 0 "J46" H 4878 6076 50  0000 L CNN
 F 1 "Conn_01x03_Female" H 4878 5985 50  0001 L CNN
-F 2 "" H 4850 6050 50  0001 C CNN
+F 2 "Connector_PinHeader_2.54mm:PinHeader_1x03_P2.54mm_Vertical" H 4850 6050 50  0001 C CNN
 F 3 "~" H 4850 6050 50  0001 C CNN
 	1    4850 6050
@@
 F 0 "J47" H 6972 3228 50  0000 R CNN
 F 1 "Conn_01x03_Male" H 6972 3183 50  0001 R CNN
-F 2 "" H 7000 3250 50  0001 C CNN
+F 2 "Connector_PinHeader_2.54mm:PinHeader_1x03_P2.54mm_Vertical" H 7000 3250 50  0001 C CNN
 F 3 "~" H 7000 3250 50  0001 C CNN
 	1    7000 3250
@@
 F 0 "J48" H 6972 4278 50  0000 R CNN
 F 1 "Conn_01x03_Male" H 6972 4233 50  0001 R CNN
-F 2 "" H 7000 4300 50  0001 C CNN
+F 2 "Connector_PinHeader_2.54mm:PinHeader_1x03_P2.54mm_Vertical" H 7000 4300 50  0001 C CNN
 F 3 "~" H 7000 4300 50  0001 C CNN
 	1    7000 4300

Commit message: BOM Update
parts added to BOM, connector cleanup. Stopping point before renumbering refdes in a more intelligent way.
Parts:
- renumbered J37 to J36, J38 to J37, J39 to J38, J40 to J39, J41 to J40, J42 to J41, J43 to J42, J44 to J43, J45 to J44, J46 to J45, J47 to J46, J48 to J47, J49 to J48, J50 to J49
Changed lines of the file:
@@
 $Descr A4 11693 8268
 encoding utf-8
-Sheet 9 13
+Sheet 7 13
 Title "IO Main Board"
 Date "2020-02-25"
@@
 P 4100 2850
 AR Path="/5E2D8DA2/5E60DD2B" Ref="J?"  Part="1"
-AR Path="/5E607732/5E60DD2B" Ref="J38"  Part="1"
-F 0 "J38" H 4028 3188 50  0000 C CNN
+AR Path="/5E607732/5E60DD2B" Ref="J37"  Part="1"
+F 0 "J37" H 4028 3188 50  0000 C CNN
 F 1 "Conn_Coaxial_x2" H 4028 3097 50  0001 C CNN
 F 2 "" H 4100 2750 50  0001 C CNN
@@
 $EndComp
 $Comp
-L Connector:Conn_01x03_Female J43
+L Connector:Conn_01x03_Female J42
 U 1 1 5E60DD36
 P 4850 2850
-F 0 "J43" H 4878 2876 50  0000 L CNN
+F 0 "J42" H 4878 2876 50  0000 L CNN
 F 1 "Conn_01x03_Female" H 4878 2785 50  0001 L CNN
 F 2 "Connector_PinHeader_2.54mm:PinHeader_1x03_P2.54mm_Vertical" H 4850 2850 50  0001 C CNN
@@
 P 4100 1800
 AR Path="/5E2D8DA2/6431D3FD" Ref="J?"  Part="1"
-AR Path="/5E607732/6431D3FD" Ref="J37"  Part="1"
-F 0 "J37" H 4028 2138 50  0000 C CNN
+AR Path="/5E607732/6431D3FD" Ref="J36"  Part="1"
+F 0 "J36" H 4028 2138 50  0000 C CNN
 F 1 "Conn_Coaxial_x2" H 4028 2047 50  0001 C CNN
 F 2 "" H 4100 1700 50  0001 C CNN
@@
 $EndComp
 $Comp
-L Connector:Conn_01x03_Female J42
+L Connector:Conn_01x03_Female J41
 U 1 1 6431D407
 P 4850 1800
-F 0 "J42" H 4878 1826 50  0000 L CNN
+F 0 "J41" H 4878 1826 50  0000 L CNN
 F 1 "Conn_01x03_Female" H 4878 1735 50  0001 L CNN
 F 2 "Connector_PinHeader_2.54mm:PinHeader_1x03_P2.54mm_Vertical" H 4850 1800 50  0001 C CNN
@@
 P 4100 4950
 AR Path="/5E2D8DA2/6433171F" Ref="J?"  Part="1"
-AR Path="/5E607732/6433171F" Ref="J40"  Part="1"
-F 0 "J40" H 4028 5288 50  0000 C CNN
+AR Path="/5E607732/6433171F" Ref="J39"  Part="1"
+F 0 "J39" H 4028 5288 50  0000 C CNN
 F 1 "Conn_Coaxial_x2" H 4028 5197 50  0001 C CNN
 F 2 "" H 4100 4850 50  0001 C CNN
@@
 $EndComp
 $Comp
-L Connector:Conn_01x03_Female J45
+L Connector:Conn_01x03_Female J44
 U 1 1 64331729
 P 4850 4950
-F 0 "J45" H 4878 4976 50  0000 L CNN
+F 0 "J44" H 4878 4976 50  0000 L CNN
 F 1 "Conn_01x03_Female" H 4878 4885 50  0001 L CNN
 F 2 "Connector_PinHeader_2.54mm:PinHeader_1x03_P2.54mm_Vertical" H 4850 4950 50  0001 C CNN
@@
 P 4100 3900
 AR Path="/5E2D8DA2/64331754" Ref="J?"  Part="1"
-AR Path="/5E607732/64331754" Ref="J39"  Part="1"
-F 0 "J39" H 4028 4238 50  0000 C CNN
+AR Path="/5E607732/64331754" Ref="J38"  Part="1"
+F 0 "J38" H 4028 4238 50  0000 C CNN
 F 1 "Conn_Coaxial_x2" H 4028 4147 50  0001 C CNN
 F 2 "" H 4100 3800 50  0001 C CNN
@@
 $EndComp
 $Comp
-L Connector:Conn_01x03_Female J44
+L Connector:Conn_01x03_Female J43
 U 1 1 6433175E
 P 4850 3900
-F 0 "J44" H 4878 3926 50  0000 L CNN
+F 0 "J43" H 4878 3926 50  0000 L CNN
 F 1 "Conn_01x03_Female" H 4878 3835 50  0001 L CNN
 F 2 "Connector_PinHeader_2.54mm:PinHeader_1x03_P2.54mm_Vertical" H 4850 3900 50  0001 C CNN
@@
 P 4100 6050
 AR Path="/5E2D8DA2/6433C001" Ref="J?"  Part="1"
-AR Path="/5E607732/6433C001" Ref="J41"  Part="1"
-F 0 "J41" H 4028 6388 50  0000 C CNN
+AR Path="/5E607732/6433C001" Ref="J40"  Part="1"
+F 0 "J40" H 4028 6388 50  0000 C CNN
 F 1 "Conn_Coaxial_x2" H 4028 6297 50  0001 C CNN
 F 2 "" H 4100 5950 50  0001 C CNN
@@
 $EndComp
 $Comp
-L Connector:Conn_01x03_Female J46
+L Connector:Conn_01x03_Female J45
 U 1 1 6433C00B
 P 4850 6050
-F 0 "J46" H 4878 6076 50  0000 L CNN
+F 0 "J45" H 4878 6076 50  0000 L CNN
 F 1 "Conn_01x03_Female" H 4878 5985 50  0001 L CNN
 F 2 "Connector_PinHeader_2.54mm:PinHeader_1x03_P2.54mm_Vertical" H 4850 6050 50  0001 C CNN
@@
 P 7750 4300
 AR Path="/5E2D8DA2/64358093" Ref="J?"  Part="1"
-AR Path="/5E607732/64358093" Ref="J50"  Part="1"
-F 0 "J50" H 7678 4638 50  0000 C CNN
+AR Path="/5E607732/64358093" Ref="J49"  Part="1"
+F 0 "J49" H 7678 4638 50  0000 C CNN
 F 1 "Conn_Coaxial_x2" H 7678 4547 50  0001 C CNN
 F 2 "" H 7750 4200 50  0001 C CNN
@@
 P 7750 3250
 AR Path="/5E2D8DA2/64354C54" Ref="J?"  Part="1"
-AR Path="/5E607732/64354C54" Ref="J49"  Part="1"
-F 0 "J49" H 7678 3588 50  0000 C CNN
+AR Path="/5E607732/64354C54" Ref="J48"  Part="1"
+F 0 "J48" H 7678 3588 50  0000 C CNN
 F 1 "Conn_Coaxial_x2" H 7678 3497 50  0001 C CNN
 F 2 "" H 7750 3150 50  0001 C CNN
@@
 $EndComp
 $Comp
-L Connector:Conn_01x03_Male J47
+L Connector:Conn_01x03_Male J46
 U 1 1 6436D21D
 P 7000 3250
-F 0 "J47" H 6972 3228 50  0000 R CNN
+F 0 "J46" H 6972 3228 50  0000 R CNN
 F 1 "Conn_01x03_Male" H 6972 3183 50  0001 R CNN
 F 2 "Connector_PinHeader_2.54mm:PinHeader_1x03_P2.54mm_Vertical" H 7000 3250 50  0001 C CNN
@@
 $EndComp
 $Comp
-L Connector:Conn_01x03_Male J48
+L Connector:Conn_01x03_Male J47
 U 1 1 6437A2AD
 P 7000 4300
-F 0 "J48" H 6972 4278 50  0000 R CNN
+F 0 "J47" H 6972 4278 50  0000 R CNN
 F 1 "Conn_01x03_Male" H 6972 4233 50  0001 R CNN
 F 2 "Connector_PinHeader_2.54mm:PinHeader_1x03_P2.54mm_Vertical" H 7000 4300 50  0001 C CNN
@@
 P 4550 1800
 AR Path="/5E26F6FE/64B8A4E5" Ref="#PWR?"  Part="1"
-AR Path="/5E607732/64B8A4E5" Ref="#PWR052"  Part="1"
-F 0 "#PWR052" H 4550 1550 50  0001 C CNN
+AR Path="/5E607732/64B8A4E5" Ref="#PWR040"  Part="1"
+F 0 "#PWR040" H 4550 1550 50  0001 C CNN
 F 1 "GND" H 4555 1627 50  0000 C CNN
 F 2 "" H 4550 1800 50  0001 C CNN
@@
 P 4550 2850
 AR Path="/5E26F6FE/64B99929" Ref="#PWR?"  Part="1"
-AR Path="/5E607732/64B99929" Ref="#PWR053"  Part="1"
-F 0 "#PWR053" H 4550 2600 50  0001 C CNN
+AR Path="/5E607732/64B99929" Ref="#PWR041"  Part="1"
+F 0 "#PWR041" H 4550 2600 50  0001 C CNN
 F 1 "GND" H 4555 2677 50  0000 C CNN
 F 2 "" H 4550 2850 50  0001 C CNN
@@
 P 4550 3900
 AR Path="/5E26F6FE/64B9AE8F" Ref="#PWR?"  Part="1"
-AR Path="/5E607732/64B9AE8F" Ref="#PWR054"  Part="1"
-F 0 "#PWR054" H 4550 3650 50  0001 C CNN
+AR Path="/5E607732/64B9AE8F" Ref="#PWR042"  Part="1"
+F 0 "#PWR042" H 4550 3650 50  0001 C CNN
 F 1 "GND" H 4555 3727 50  0000 C CNN
 F 2 "" H 4550 3900 50  0001 C CNN
@@
 P 4550 6050
 AR Path="/5E26F6FE/64B9C67B" Ref="#PWR?"  Part="1"
-AR Path="/5E607732/64B9C67B" Ref="#PWR056"  Part="1"
-F 0 "#PWR056" H 4550 5800 50  0001 C CNN
+AR Path="/5E607732/64B9C67B" Ref="#PWR044"  Part="1"
+F 0 "#PWR044" H 4550 5800 50  0001 C CNN
 F 1 "GND" H 4555 5877 50  0000 C CNN
 F 2 "" H 4550 6050 50  0001 C CNN
@@
 P 4550 4950
 AR Path="/5E26F6FE/64B9F2DA" Ref="#PWR?"  Part="1"
-AR Path="/5E607732/64B9F2DA" Ref="#PWR055"  Part="1"
-F 0 "#PWR055" H 4550 4700 50  0001 C CNN
+AR Path="/5E607732/64B9F2DA" Ref="#PWR043"  Part="1"
+F 0 "#PWR043" H 4550 4700 50  0001 C CNN
 F 1 "GND" H 4555 4777 50  0000 C CNN
 F 2 "" H 4550 4950 50  0001 C CNN
@@
 P 7300 3250
 AR Path="/5E26F6FE/64BA0A7B" Ref="#PWR?"  Part="1"
-AR Path="/5E607732/64BA0A7B" Ref="#PWR057"  Part="1"
-F 0 "#PWR057" H 7300 3000 50  0001 C CNN
+AR Path="/5E607732/64BA0A7B" Ref="#PWR045"  Part="1"
+F 0 "#PWR045" H 7300 3000 50  0001 C CNN
 F 1 "GND" H 7305 3077 50  0000 C CNN
 F 2 "" H 7300 3250 50  0001 C CNN
@@
 P 7300 4300
 AR Path="/5E26F6FE/64BA2069" Ref="#PWR?"  Part="1"
-AR Path="/5E607732/64BA2069" Ref="#PWR058"  Part="1"
-F 0 "#PWR058" H 7300 4050 50  0001 C CNN
+AR Path="/5E607732/64BA2069" Ref="#PWR046"  Part="1"
+F 0 "#PWR046" H 7300 4050 50  0001 C CNN
 F 1 "GND" H 7305 4127 50  0000 C CNN
 F 2 "" H 7300 4300 50  0001 C CNN
@@
 P 4100 6350
 AR Path="/5E26F6FE/64BAD508" Ref="#PWR?"  Part="1"
-AR Path="/5E607732/64BAD508" Ref="#PWR051"  Part="1"
-F 0 "#PWR051" H 4100 6100 50  0001 C CNN
+AR Path="/5E607732/64BAD508" Ref="#PWR039"  Part="1"
+F 0 "#PWR039" H 4100 6100 50  0001 C CNN
 F 1 "GND" H 4105 6177 50  0000 C CNN
 F 2 "" H 4100 6350 50  0001 C CNN
@@
 P 4100 5250
 AR Path="/5E26F6FE/64BAEC2E" Ref="#PWR?"  Part="1"
-AR Path="/5E607732/64BAEC2E" Ref="#PWR050"  Part="1"
-F 0 "#PWR050" H 4100 5000 50  0001 C CNN
+AR Path="/5E607732/64BAEC2E" Ref="#PWR038"  Part="1"
+F 0 "#PWR038" H 4100 5000 50  0001 C CNN
 F 1 "GND" H 4105 5077 50  0000 C CNN
 F 2 "" H 4100 5250 50  0001 C CNN
@@
 P 4100 4200
 AR Path="/5E26F6FE/64BB01CD" Ref="#PWR?"  Part="1"
-AR Path="/5E607732/64BB01CD" Ref="#PWR049"  Part="1"
-F 0 "#PWR049" H 4100 3950 50  0001 C CNN
+AR Path="/5E607732/64BB01CD" Ref="#PWR037"  Part="1"
+F 0 "#PWR037" H 4100 3950 50  0001 C CNN
 F 1 "GND" H 4105 4027 50  0000 C CNN
 F 2 "" H 4100 4200 50  0001 C CNN
@@
 P 4100 3150
 AR Path="/5E26F6FE/64BB1739" Ref="#PWR?"  Part="1"
-AR Path="/5E607732/64BB1739" Ref="#PWR048"  Part="1"
-F 0 "#PWR048" H 4100 2900 50  0001 C CNN
+AR Path="/5E607732/64BB1739" Ref="#PWR036"  Part="1"
+F 0 "#PWR036" H 4100 2900 50  0001 C CNN
 F 1 "GND" H 4105 2977 50  0000 C CNN
 F 2 "" H 4100 3150 50  0001 C CNN
@@
 P 4100 2100
 AR Path="/5E26F6FE/64BB2C61" Ref="#PWR?"  Part="1"
-AR Path="/5E607732/64BB2C61" Ref="#PWR047"  Part="1"
-F 0 "#PWR047" H 4100 1850 50  0001 C CNN
+AR Path="/5E607732/64BB2C61" Ref="#PWR035"  Part="1"
+F 0 "#PWR035" H 4100 1850 50  0001 C CNN
 F 1 "GND" H 4105 1927 50  0000 C CNN
 F 2 "" H 4100 2100 50  0001 C CNN
@@
 P 7750 3550
 AR Path="/5E26F6FE/64BB4167" Ref="#PWR?"  Part="1"
-AR Path="/5E607732/64BB4167" Ref="#PWR059"  Part="1"
-F 0 "#PWR059" H 7750 3300 50  0001 C CNN
+AR Path="/5E607732/64BB4167" Ref="#PWR047"  Part="1"
+F 0 "#PWR047" H 7750 3300 50  0001 C CNN
 F 1 "GND" H 7755 3377 50  0000 C CNN
 F 2 "" H 7750 3550 50  0001 C CNN
@@
 P 7750 4600
 AR Path="/5E26F6FE/64BB6E12" Ref="#PWR?"  Part="1"
-AR Path="/5E607732/64BB6E12" Ref="#PWR060"  Part="1"
-F 0 "#PWR060" H 7750 4350 50  0001 C CNN
+AR Path="/5E607732/64BB6E12" Ref="#PWR048"  Part="1"
+F 0 "#PWR048" H 7750 4350 50  0001 C CNN
 F 1 "GND" H 7755 4427 50  0000 C CNN
 F 2 "" H 7750 4600 50  0001 C CNN
