File: preamp-layout/preamp-kicad/+-15V_PWR_SUPPLY.sch (KiCad schematic (older format))
At the start: 33 parts, among them J10 Conn_01x03_Male, J11 Conn_01x03_Male, J8 Screw_Terminal_01x03, J9 Conn_01x03_Male, T1 Transformer_1P_2S, U1 LM7805, U2 LM7905

Commit message: Footprint assignment updates
Parts:
- C10, C11: footprint (none) -> Capacitor_THT:CP_Radial_D6.3mm_P2.50mm
- C2, C3, C4, C5: footprint (none) -> Capacitor_THT:CP_Radial_D12.5mm_P5.00mm
- R4, R5: footprint (none) -> Resistor_THT:R_Axial_DIN0414_L11.9mm_D4.5mm_P15.24mm_Horizontal
- R6, R7: footprint (none) -> Resistor_SMD:R_1206_3216Metric_Pad1.42x1.75mm_HandSolder
- U1: footprint (none) -> Package_TO_SOT_THT:TO-220-3_Vertical
Changed lines of the file:
@@
 F 0 "R6" H 8370 2996 50  0000 L CNN
 F 1 "240R" H 8370 2905 50  0000 L CNN
-F 2 "" V 8230 2950 50  0001 C CNN
+F 2 "Resistor_SMD:R_1206_3216Metric_Pad1.42x1.75mm_HandSolder" V 8230 2950 50  0001 C CNN
 F 3 "~" H 8300 2950 50  0001 C CNN
 	1    8300 2950
@@
 F 0 "R4" V 5893 2350 50  0000 C CNN
 F 1 "10R 1W" V 5984 2350 50  0000 C CNN
-F 2 "" V 6030 2350 50  0001 C CNN
+F 2 "Resistor_THT:R_Axial_DIN0414_L11.9mm_D4.5mm_P15.24mm_Horizontal" V 6030 2350 50  0001 C CNN
 F 3 "~" H 6100 2350 50  0001 C CNN
 	1    6100 2350
@@
 F 0 "C2" H 5815 3096 50  0000 L CNN
 F 1 "2200uF" H 5815 3005 50  0000 L CNN
-F 2 "" H 5700 3050 50  0001 C CNN
+F 2 "Capacitor_THT:CP_Radial_D12.5mm_P5.00mm" H 5700 3050 50  0001 C CNN
 F 3 "~" H 5700 3050 50  0001 C CNN
 	1    5700 3050
@@
 F 0 "C4" H 6615 3096 50  0000 L CNN
 F 1 "2200uF" H 6615 3005 50  0000 L CNN
-F 2 "" H 6500 3050 50  0001 C CNN
+F 2 "Capacitor_THT:CP_Radial_D12.5mm_P5.00mm" H 6500 3050 50  0001 C CNN
 F 3 "~" H 6500 3050 50  0001 C CNN
 	1    6500 3050
@@
 F 0 "C10" H 10015 2996 50  0000 L CNN
 F 1 "100uF" H 10015 2905 50  0000 L CNN
-F 2 "" H 9900 2950 50  0001 C CNN
+F 2 "Capacitor_THT:CP_Radial_D6.3mm_P2.50mm" H 9900 2950 50  0001 C CNN
 F 3 "~" H 9900 2950 50  0001 C CNN
 	1    9900 2950
@@
 F 0 "U1" H 7800 2592 50  0000 C CNN
 F 1 "LM7805" H 7800 2501 50  0000 C CNN
-F 2 "" H 7825 2200 50  0001 L CIN
+F 2 "Package_TO_SOT_THT:TO-220-3_Vertical" H 7825 2200 50  0001 L CIN
 F 3 "http://www.st.com/content/ccc/resource/technical/document/datasheet/41/4f/b3/b0/12/d4/47/88/CD00000444.pdf/files/CD00000444.pdf/jcr:content/translations/en.CD00000444.pdf" H 7800 2300 50  0001 C CNN
 	1    7800 2350
@@
 F 0 "R7" H 8370 4104 50  0000 L CNN
 F 1 "240R" H 8370 4195 50  0000 L CNN
-F 2 "" V 8230 4150 50  0001 C CNN
+F 2 "Resistor_SMD:R_1206_3216Metric_Pad1.42x1.75mm_HandSolder" V 8230 4150 50  0001 C CNN
 F 3 "~" H 8300 4150 50  0001 C CNN
 	1    8300 4150
@@
 F 0 "R5" V 6307 4750 50  0000 C CNN
 F 1 "10R 1W" V 6216 4750 50  0000 C CNN
-F 2 "" V 6030 4750 50  0001 C CNN
+F 2 "Resistor_THT:R_Axial_DIN0414_L11.9mm_D4.5mm_P15.24mm_Horizontal" V 6030 4750 50  0001 C CNN
 F 3 "~" H 6100 4750 50  0001 C CNN
 	1    6100 4750
@@
 F 0 "C3" H 5815 4096 50  0000 L CNN
 F 1 "2200uF" H 5815 4005 50  0000 L CNN
-F 2 "" H 5700 4050 50  0001 C CNN
+F 2 "Capacitor_THT:CP_Radial_D12.5mm_P5.00mm" H 5700 4050 50  0001 C CNN
 F 3 "~" H 5700 4050 50  0001 C CNN
 	1    5700 4050
@@
 F 0 "C5" H 6615 4096 50  0000 L CNN
 F 1 "2200uF" H 6615 4005 50  0000 L CNN
-F 2 "" H 6500 4050 50  0001 C CNN
+F 2 "Capacitor_THT:CP_Radial_D12.5mm_P5.00mm" H 6500 4050 50  0001 C CNN
 F 3 "~" H 6500 4050 50  0001 C CNN
 	1    6500 4050
@@
 F 0 "C11" H 9785 4196 50  0000 R CNN
 F 1 "100uF" H 9785 4105 50  0000 R CNN
-F 2 "" H 9900 4150 50  0001 C CNN
+F 2 "Capacitor_THT:CP_Radial_D6.3mm_P2.50mm" H 9900 4150 50  0001 C CNN
 F 3 "~" H 9900 4150 50  0001 C CNN
 	1    9900 4150

Commit message: voltage regulator update
regulators used in 15V supply changed from LM7805, LM7905 to LM7815, LM7915
Parts:
- U1: value LM7805 -> LM7815
- U2: value LM7905 -> LM7915
Changed lines of the file:
@@
 AR Path="/5E27B612/5FE3F8F2" Ref="U1"  Part="1"
 F 0 "U1" H 7800 2592 50  0000 C CNN
-F 1 "LM7805" H 7800 2501 50  0000 C CNN
+F 1 "LM7815" H 7800 2501 50  0000 C CNN
 F 2 "Package_TO_SOT_THT:TO-220-3_Vertical" H 7825 2200 50  0001 L CIN
 F 3 "http://www.st.com/content/ccc/resource/technical/document/datasheet/41/4f/b3/b0/12/d4/47/88/CD00000444.pdf/files/CD00000444.pdf/jcr:content/translations/en.CD00000444.pdf" H 7800 2300 50  0001 C CNN
@@
 AR Path="/5E27B612/5FE3F8FA" Ref="U2"  Part="1"
 F 0 "U2" H 7800 4601 50  0000 C CNN
-F 1 "LM7905" H 7800 4510 50  0000 C CNN
+F 1 "LM7915" H 7800 4510 50  0000 C CNN
 F 2 "Package_TO_SOT_THT:TO-220-3_Vertical" H 7800 4550 50  0001 C CIN
 F 3 "http://www.fairchildsemi.com/ds/LM/LM7905.pdf" H 7800 4750 50  0001 C CNN

Commit message: balanced IO update
other general minor updates
Changed lines of the file:
@@
 Wire Wire Line
 	9900 3100 9900 3550
-Text GLabel 10150 2350 2    50   UnSpc ~ 0
+Text GLabel 9900 2100 1    50   UnSpc ~ 0
 +15V
 Text Label 5500 4750 2    50   ~ 0
@@
 Wire Wire Line
 	9900 4000 9900 3550
-Text GLabel 10150 4750 2    50   UnSpc ~ 0
+Text GLabel 9900 5000 3    50   UnSpc ~ 0
 -15V
 $Comp
@@
 Connection ~ 9900 3550
 Wire Wire Line
-	9900 2350 10150 2350
+	9900 2350 9900 2100
 Connection ~ 9900 4750
 Wire Wire Line
-	9900 4750 10150 4750
+	9900 4750 9900 5000
 $EndSCHEMATC
