File: preamp-layout/preamp-kicad/preamp.kicad_pcb (KiCad board)
At the start: 2 copper layers, 324 parts, among them J10 Conn_01x03_Male, J11 Conn_01x03_Male, J12 Conn_01x02_Male, J13 Conn_01x02_Male, J14 Conn_01x02_Male, J15 Screw_Terminal_01x03, J16 Conn_01x03_Female, J17 Conn_01x03_Female, J18 Conn_01x03_Female, J19 Conn_01x03_Female, J2 Screw_Terminal_01x03, J20 Conn_01x03_Female, J21 Conn_01x03_Female, J22 Conn_01x03_Female, J23 Conn_01x03_Female, J25 Conn_01x02_Male, J26 Conn_01x02_Male, J27 Conn_01x15_Female, J28 Conn_01x15_Female, J29 Conn_01x06_Female, J3 Conn_01x02_Female, J30 Conn_01x03_Female, J31 Conn_01x03_Female, J32 Conn_01x03_Female, J33 Conn_01x03_Male, J34 Conn_01x02_Male, J35 Conn_01x02_Male, J4 Conn_01x02_Male, J41 Conn_01x03_Female, J42 Conn_01x03_Female, J43 Conn_01x03_Female, J44 Conn_01x03_Female, J45 Conn_01x03_Female, J46 Conn_01x03_Male, J47 Conn_01x03_Male, J5 Screw_Terminal_01x03, J50 Conn_01x03_Female, J51 Conn_01x03_Male, J52 Conn_01x03_Male, J53 Conn_01x03_Male, J54 Conn_01x03_Male, J57 Conn_01x03_Male, J58 Conn_01x03_Male, J59 Conn_01x03_Female, J6 Conn_01x02_Female, J60 Conn_01x02_Male, J61 Conn_01x02_Male, J62 Conn_01x03_Female, J63 Conn_01x03_Female, J64 Conn_01x05_Male, J65 Conn_01x02_Male, J66 Conn_01x02_Male, J67 Conn_01x03_Female, J68 Conn_01x03_Female, J69 Conn_01x03_Male, J7 Screw_Terminal_01x03, J70 Conn_01x03_Male, J71 Conn_01x03_Male, J72 Conn_01x04_Male, J73 Conn_01x03_Male, J74 Conn_01x03_Male, J75 Conn_01x03_Male, J76 Conn_01x03_Female, J77 Conn_01x04_Female, J78 Conn_01x04_Female, J79 Conn_01x04_Male, J8 Screw_Terminal_01x03, J84 Conn_01x03_Male, J85 Conn_01x03_Male, J86 Conn_01x03_Female, J87 Conn_01x03_Male, J9 Conn_01x03_Male, K2 G6JU, K3 G6JU, K4 G6JU, K5 G6JU, K6 G6JU, K7 G6JU, K8 G6JU, U1 LM7815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

Commit message: MCU cleanup
removed separate header schematic symbols for MCU mounting because that was dumb. Updated ESP32 footprint. Played around with pcb layout even though I'm not close to ready for that yet, just wanted to mess around. Added pinouts for ESP32 / ESP8266.
Parts:
- removed J27, J28: Conn_01x15_Female, Connector_PinHeader_2.54mm:PinHeader_1x15_P2.54mm_Vertical
- removed J29: Conn_01x06_Female, Connector_PinHeader_2.54mm:PinHeader_1x06_P2.54mm_Vertical
- removed J30, J31, J32, J50, J76: Conn_01x03_Female, Connector_PinHeader_2.54mm:PinHeader_1x03_P2.54mm_Vertical
- removed J57: Conn_01x03_Male, Connector_PinHeader_2.54mm:PinHeader_1x03_P2.54mm_Vertical
- removed U9: MCP4902, Package_SO:SOIC-14_3.9x8.7mm_P1.27mm
- added C100: 100nF, Capacitor_SMD:C_0805_2012Metric_Pad1.15x1.40mm_HandSolder, F.Cu at (-133.1, 163.7)
- added C101: 100nF, Capacitor_SMD:C_0805_2012Metric_Pad1.15x1.40mm_HandSolder, F.Cu at (-115.9, 146.8)
- added C102: 100nF, Capacitor_SMD:C_0805_2012Metric_Pad1.15x1.40mm_HandSolder, F.Cu at (-99.0, 130.6)
- added C103: 100nF, Capacitor_SMD:C_0805_2012Metric_Pad1.15x1.40mm_HandSolder, F.Cu at (-124.3, 153.4)
- added C104: 100nF, Capacitor_SMD:C_0805_2012Metric_Pad1.15x1.40mm_HandSolder, F.Cu at (-107.5, 137.3)
- added C105: 100nF, Capacitor_SMD:C_0805_2012Metric_Pad1.15x1.40mm_HandSolder, F.Cu at (-115.9, 143.9)
- added C106: 100nF, Capacitor_SMD:C_0805_2012Metric_Pad1.15x1.40mm_HandSolder, F.Cu at (-137.9, 163.7)
- added C107: 100nF, Capacitor_SMD:C_0805_2012Metric_Pad1.15x1.40mm_HandSolder, F.Cu at (-124.3, 150.5)
- added C108: 100nF, Capacitor_SMD:C_0805_2012Metric_Pad1.15x1.40mm_HandSolder, F.Cu at (-110.0, 152.7)
- added C109: 100nF, Capacitor_SMD:C_0805_2012Metric_Pad1.15x1.40mm_HandSolder, F.Cu at (-99.0, 133.6)
- added C110: 100nF, Capacitor_SMD:C_0805_2012Metric_Pad1.15x1.40mm_HandSolder, F.Cu at (110.7, 116.9)
- added C111: 100nF, Capacitor_SMD:C_0805_2012Metric_Pad1.15x1.40mm_HandSolder, F.Cu at (-111.1, 146.8)
- added C112: 100nF, Capacitor_SMD:C_0805_2012Metric_Pad1.15x1.40mm_HandSolder, F.Cu at (-124.3, 159.3)
- added C113: 100nF, Capacitor_SMD:C_0805_2012Metric_Pad1.15x1.40mm_HandSolder, F.Cu at (-114.8, 149.8)
- added C114: 100nF, Capacitor_SMD:C_0805_2012Metric_Pad1.15x1.40mm_HandSolder, F.Cu at (-128.4, 163.7)
- added C115: 100nF, Capacitor_SMD:C_0805_2012Metric_Pad1.15x1.40mm_HandSolder, F.Cu at (-102.7, 140.2)
- added C116: 100nF, Capacitor_SMD:C_0805_2012Metric_Pad1.15x1.40mm_HandSolder, F.Cu at (-106.4, 143.2)
- added C117: 100nF, Capacitor_SMD:C_0805_2012Metric_Pad1.15x1.40mm_HandSolder, F.Cu at (-98.0, 136.5)
- added C118: 100nF, Capacitor_SMD:C_0805_2012Metric_Pad1.15x1.40mm_HandSolder, F.Cu at (-114.8, 152.7)
- added C119: 100nF, Capacitor_SMD:C_0805_2012Metric_Pad1.15x1.40mm_HandSolder, F.Cu at (110.7, 119.9)
- added C120: 0.1uF, Capacitor_SMD:C_0805_2012Metric_Pad1.15x1.40mm_HandSolder, F.Cu at (264.4, 72.3)
- added C121: 0.1uF, Capacitor_SMD:C_0805_2012Metric_Pad1.15x1.40mm_HandSolder, F.Cu at (258.5, 78.6)
- added C122: 0.1uF, Capacitor_SMD:C_0805_2012Metric_Pad1.15x1.40mm_HandSolder, F.Cu at (167.1, 153.1)
- added C41: 0.1uF, Capacitor_SMD:C_0805_2012Metric_Pad1.15x1.40mm_HandSolder, F.Cu at (258.5, 69.8)
- added C42: 0.1uF, Capacitor_SMD:C_0805_2012Metric_Pad1.15x1.40mm_HandSolder, F.Cu at (264.5, 63.5)
- added C43: 0.1uF, Capacitor_SMD:C_0805_2012Metric_Pad1.15x1.40mm_HandSolder, F.Cu at (268.1, 60.2)
- added C44: 0.1uF, Capacitor_SMD:C_0805_2012Metric_Pad1.15x1.40mm_HandSolder, F.Cu at (254.9, 73.2)
- added C61: 0.1uF, Capacitor_SMD:C_0805_2012Metric_Pad1.15x1.40mm_HandSolder, F.Cu at (259.7, 72.7)
- added C62: 0.1uF, Capacitor_SMD:C_0805_2012Metric_Pad1.15x1.40mm_HandSolder, F.Cu at (263.3, 69.4)
- added C73: 22uF, Capacitor_SMD:C_0805_2012Metric_Pad1.15x1.40mm_HandSolder, F.Cu at (210.9, 150.0)
- added C74: 22uF, Capacitor_SMD:C_0805_2012Metric_Pad1.15x1.40mm_HandSolder, F.Cu at (225.2, 139.8)
- added C75: 0.1uF, Capacitor_SMD:C_0805_2012Metric_Pad1.15x1.40mm_HandSolder, F.Cu at (5.08, -56.5)
- added C76: 0.1uF, Capacitor_SMD:C_0805_2012Metric_Pad1.15x1.40mm_HandSolder, F.Cu at (-27.3, -55.2)
- added C77: 0.1uF, Capacitor_SMD:C_0805_2012Metric_Pad1.15x1.40mm_HandSolder, F.Cu at (165.4, 142.0)
- added C78: 0.1uF, Capacitor_SMD:C_0805_2012Metric_Pad1.15x1.40mm_HandSolder, F.Cu at (165.4, 139.0)
- added C79: 0.1uF, Capacitor_SMD:C_0805_2012Metric_Pad1.15x1.40mm_HandSolder, F.Cu at (126.5, 129.7)
- added C80: 100nF, Capacitor_SMD:C_0805_2012Metric_Pad1.15x1.40mm_HandSolder, F.Cu at (-101.6, 143.2)
- added C81: 100nF, Capacitor_SMD:C_0805_2012Metric_Pad1.15x1.40mm_HandSolder, F.Cu at (-98.0, 139.5)
- added C82: 100nF, Capacitor_SMD:C_0805_2012Metric_Pad1.15x1.40mm_HandSolder, F.Cu at (-110.0, 149.8)
- added C83: 100nF, Capacitor_SMD:C_0805_2012Metric_Pad1.15x1.40mm_HandSolder, F.Cu at (-123.6, 162.3)
- added C84: 100nF, Capacitor_SMD:C_0805_2012Metric_Pad1.15x1.40mm_HandSolder, F.Cu at (-119.5, 159.3)
- added C85: 100nF, Capacitor_SMD:C_0805_2012Metric_Pad1.15x1.40mm_HandSolder, F.Cu at (-106.4, 146.1)
- added C86: 100nF, Capacitor_SMD:C_0805_2012Metric_Pad1.15x1.40mm_HandSolder, F.Cu at (-114.8, 155.7)
- added C87: 100nF, Capacitor_SMD:C_0805_2012Metric_Pad1.15x1.40mm_HandSolder, F.Cu at (-119.5, 156.4)
- added C88: 100nF, Capacitor_SMD:C_0805_2012Metric_Pad1.15x1.40mm_HandSolder, F.Cu at (-142.6, 163.7)
- added C89: 100nF, Capacitor_SMD:C_0805_2012Metric_Pad1.15x1.40mm_HandSolder, F.Cu at (-147.4, 163.7)
- added C90: 100nF, Capacitor_SMD:C_0805_2012Metric_Pad1.15x1.40mm_HandSolder, F.Cu at (-166.4, 163.7)
- added C91: 100nF, Capacitor_SMD:C_0805_2012Metric_Pad1.15x1.40mm_HandSolder, F.Cu at (-161.6, 163.7)
- added C92: 100nF, Capacitor_SMD:C_0805_2012Metric_Pad1.15x1.40mm_HandSolder, F.Cu at (-156.9, 163.7)
- added C93: 100nF, Capacitor_SMD:C_0805_2012Metric_Pad1.15x1.40mm_HandSolder, F.Cu at (-152.1, 163.7)
- added C94: 100nF, Capacitor_SMD:C_0805_2012Metric_Pad1.15x1.40mm_HandSolder, F.Cu at (-119.5, 153.4)
- added C95: 100nF, Capacitor_SMD:C_0805_2012Metric_Pad1.15x1.40mm_HandSolder, F.Cu at (-102.7, 137.3)
- added C96: 100nF, Capacitor_SMD:C_0805_2012Metric_Pad1.15x1.40mm_HandSolder, F.Cu at (-111.1, 143.9)
- added C97: 100nF, Capacitor_SMD:C_0805_2012Metric_Pad1.15x1.40mm_HandSolder, F.Cu at (-107.5, 140.2)
- added C98: 100nF, Capacitor_SMD:C_0805_2012Metric_Pad1.15x1.40mm_HandSolder, F.Cu at (-124.3, 156.4)
- added C99: 100nF, Capacitor_SMD:C_0805_2012Metric_Pad1.15x1.40mm_HandSolder, F.Cu at (-119.5, 150.5)
- added J24: Conn_01x05_Female, Connector_PinHeader_2.54mm:PinHeader_1x05_P2.54mm_Vertical, F.Cu at (131.9, 150.6)
- added J55: Conn_01x03_Male, Connector_PinHeader_2.54mm:PinHeader_1x03_P2.54mm_Vertical, F.Cu at (144.2, 135.8)
- added R122: 1k, Resistor_SMD:R_1206_3216Metric_Pad1.42x1.75mm_HandSolder, F.Cu at (155.8, 155.8)
- added R123: 1k, Resistor_SMD:R_1206_3216Metric_Pad1.42x1.75mm_HandSolder, F.Cu at (151.4, 159.7)
- added R124: 1k, Resistor_SMD:R_1206_3216Metric_Pad1.42x1.75mm_HandSolder, F.Cu at (165.4, 150.0)
- added R125: 1k, Resistor_SMD:R_1206_3216Metric_Pad1.42x1.75mm_HandSolder, F.Cu at (141.9, 165.5)
- added R134: 10k, Resistor_SMD:R_1206_3216Metric_Pad1.42x1.75mm_HandSolder, F.Cu at (137.2, 169.4)
- added R64: 5.1k, Resistor_SMD:R_1206_3216Metric_Pad1.42x1.75mm_HandSolder, F.Cu at (260.6, 53.8)
- added R65: 5.1k, Resistor_SMD:R_1206_3216Metric_Pad1.42x1.75mm_HandSolder, F.Cu at (264.2, 50.5)
- added R66: 5.1k, Resistor_SMD:R_1206_3216Metric_Pad1.42x1.75mm_HandSolder, F.Cu at (247.2, 66.9)
- added R67: 5.1k, Resistor_SMD:R_1206_3216Metric_Pad1.42x1.75mm_HandSolder, F.Cu at (250.8, 63.5)
- added R68: 100k, Resistor_SMD:R_1206_3216Metric_Pad1.42x1.75mm_HandSolder, F.Cu at (230.5, 130.4)
- added R69: 100k, Resistor_SMD:R_1206_3216Metric_Pad1.42x1.75mm_HandSolder, F.Cu at (224.5, 133.8)
- added R70: 1k, Resistor_SMD:R_1206_3216Metric_Pad1.42x1.75mm_HandSolder, F.Cu at (149.1, 169.5)
- added R71: 1k, Resistor_SMD:R_1206_3216Metric_Pad1.42x1.75mm_HandSolder, F.Cu at (157.4, 162.4)
- added U19: MCP23017_SO, Package_SO:SOIC-28W_7.5x17.9mm_P1.27mm, F.Cu at (-18.6, -58.1)
- added U4: MCP23017_SO, Package_SO:SOIC-28W_7.5x17.9mm_P1.27mm, F.Cu at (123.1, 158.0)
- added U5: ESP32-DevKitC, preamp:ESP32_MELIFE_DEVKIT, F.Cu at (-80.0, -73.7)
- J64: value Conn_01x05_Male -> Conn_01x02_Male; footprint Connector_PinHeader_2.54mm:PinHeader_1x05_P2.54mm_Vertical -> Connector_JST:JST_EH_B2B-EH-A_1x02_P2.50mm_Vertical
- R110, R111, R93, R94: value 1k -> 909R
- R74, R75: value 500R -> 499R
- U10: value MCP4902 -> TCA9548APWR; footprint Package_SO:SOIC-14_3.9x8.7mm_P1.27mm -> Package_SO:TSSOP-24_4.4x7.8mm_P0.65mm
- U11: value TL072 -> TL074CDR; footprint Package_DIP:DIP-8_W7.62mm_Socket_LongPads -> Package_SO:SOIC-14_3.9x8.7mm_P1.27mm
- U12: value TL072 -> WeMos_D1_mini; footprint Package_DIP:DIP-8_W7.62mm_Socket_LongPads -> Module:WEMOS_D1_mini_light
- U15, U18, U21, U22, U23: value TL072 -> NJM2068M; footprint Package_DIP:DIP-8_W7.62mm_Socket_LongPads -> Package_SO:SOP-8_3.9x4.9mm_P1.27mm
- U6: value MCP23S17_SP -> MCP23017_SO; footprint Package_DIP:DIP-28_W7.62mm -> Package_SO:SOIC-28W_7.5x17.9mm_P1.27mm
- moved D2 329.3 mm to (215.3, -129.8), turned to 180 degrees
- moved J10 314.5 mm to (221.0, -120.5), turned to 270 degrees
- moved J11 310.2 mm to (221.0, -109.2), turned to 270 degrees
- moved R6 309.2 mm to (204.2, -121.4), turned to 270 degrees
- moved D3 306.1 mm to (214.8, -106.8)
- moved D6 306.1 mm to (206.8, -121.3), turned to 270 degrees
- moved R7 306.1 mm to (204.2, -114.8), turned to 90 degrees
- moved C10 305.0 mm to (214.4, -122.9), turned to 270 degrees
- moved R2 304.8 mm to (215.2, -132.2), turned to 180 degrees
- moved R4 299.4 mm to (184.8, -136.4), turned to 180 degrees
- moved R3 296.9 mm to (214.7, -104.3), turned to 180 degrees
- moved C4 294.3 mm to (184.2, -127.9), turned to 270 degrees
- moved C9 293.0 mm to (209.3, -115.3), turned to 90 degrees
- moved U2 292.9 mm to (194.1, -113.8)
- moved D7 288.6 mm to (206.8, -114.9), turned to 270 degrees
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Connections:
- net /+-15V PWR SUPPLY/AC+ renamed /+-15V PWR SUPPLY/AC_HOT
- net /+-15V PWR SUPPLY/AC- renamed /+-15V PWR SUPPLY/AC_N
- net /AC input/AC_IN_+ renamed /AC input/AC_IN_HOT
- net /AC input/PWR_SW_2 renamed /AC input/PWR_SW
- net /BAL_IN_L renamed /IO/A_IN_5_L
- net /BAL_IN_R renamed /IO/A_IN_5_R
- net /BAL_OUT_L renamed /IO/A_OUT_2_L
- net /BAL_OUT_R renamed /IO/A_OUT_2_R
- net /Volume Control/Buffered_DAC_Main_L renamed /Volume Control/DAC_CTRL_1_L
- net /Volume Control/Buffered_DAC_Main_R renamed /Volume Control/DAC_CTRL_1_R
- net /headphone amp/L_IN renamed /headphone amp/IN_L
- net /headphone amp/R_IN renamed /headphone amp/IN_R
- C31 pad 1: /Volume Control/Buffered_DAC_HP_L -> /Volume Control/DAC_CTRL_2_L
- C32 pad 1: /Volume Control/Buffered_DAC_HP_R -> /Volume Control/DAC_CTRL_2_R
- J52 pad 1: /IO/A_IN_3_L -> /IO/A_IN_2_L
- J52 pad 3: /IO/A_IN_3_R -> /IO/A_IN_2_R
- J53 pad 1: /IO/A_IN_2_L -> /IO/A_IN_3_L
- J53 pad 3: /IO/A_IN_2_R -> /IO/A_IN_3_R
- J64 pad 1: /Volume Control/CLK -> /Volume Control/DAC_SDA
- J64 pad 2: /Volume Control/~LDAC -> /Volume Control/DAC_SCL
- J69 pad 1: /input selector/A_OUT_R -> /input selector/A_OUT_L
- J69 pad 3: /input selector/A_OUT_L -> /input selector/A_OUT_R
- R103 pad 1: Net-(R103-Pad1) -> Net-(C73-Pad1)
- R106 pad 2: Net-(R103-Pad1) -> Net-(C73-Pad2)
- R119 pad 1: Net-(R119-Pad1) -> Net-(C74-Pad1)
- R121 pad 2: Net-(R119-Pad1) -> Net-(C74-Pad2)
- R35 pad 2: Net-(R35-Pad2) -> /Volume Control/DAC_A
- R36 pad 2: Net-(R36-Pad2) -> /Volume Control/DAC_B
- R37 pad 2: Net-(R37-Pad2) -> /Volume Control/DAC_C
- R38 pad 2: Net-(R38-Pad2) -> /Volume Control/DAC_D
- R49 pad 1: /Volume Control/Buffered_DAC_HP_L -> /Volume Control/DAC_CTRL_2_L
- R50 pad 1: /Volume Control/Buffered_DAC_HP_R -> /Volume Control/DAC_CTRL_2_R
- R78 pad 1: /headphone amp/L_OUT -> /headphone amp/OUT_L
- R79 pad 1: /headphone amp/R_OUT -> /headphone amp/OUT_R
- U10 pad 1: +5V -> GND
- U10 pad 10: Net-(R38-Pad2) -> Net-(R132-Pad2)
- U10 pad 11: +5V -> Net-(R133-Pad2)
- U10 pad 13: +5V -> Net-(U10-Pad13)
- U10 pad 14: Net-(R37-Pad2) -> Net-(U10-Pad14)
- U10 pad 2: Net-(U10-Pad2) -> GND
- U10 pad 3: /MCU/CS_VOL_HP -> /MCU/~I2C_RST
- U10 pad 4: /Volume Control/CLK -> /MCU/IO_SDA
- U10 pad 5: /Volume Control/MOSI -> /MCU/IO_SCL
- U10 pad 6: Net-(U10-Pad6) -> /Volume Control/DAC_SDA
- U10 pad 7: Net-(U10-Pad7) -> /Volume Control/DAC_SCL
- U10 pad 8: /Volume Control/~LDAC -> /MCU/FP_SDA
- U10 pad 9: +5V -> /MCU/FP_SCL
- U11 pad 4: -15V -> +15V
- U11 pad 8: +15V -> /Volume Control/DAC_CTRL_2_L
- U12 pad 1: /Volume Control/Buffered_DAC_HP_L -> Net-(U12-Pad1)
- U12 pad 2: Net-(C31-Pad2) -> Net-(U12-Pad2)
- U12 pad 3: GND -> Net-(U12-Pad3)
- U12 pad 4: -15V -> Net-(U12-Pad4)
- U12 pad 5: GND -> Net-(U12-Pad5)
- U12 pad 6: Net-(C32-Pad2) -> /MCU/LED_DT
- U12 pad 7: /Volume Control/Buffered_DAC_HP_R -> Net-(U12-Pad7)
- U12 pad 8: +15V -> Net-(U12-Pad8)
- U13 pad 5: -15V -> Net-(R64-Pad1)
- U13 pad 7: -15V -> +15V
- U14 pad 5: -15V -> Net-(R65-Pad1)
- U14 pad 7: -15V -> +15V
- U16 pad 2: /Volume Control/Buffered_DAC_HP_L -> /Volume Control/DAC_CTRL_2_L
- U16 pad 5: -15V -> Net-(R66-Pad1)
- U16 pad 7: -15V -> +15V
- U17 pad 2: /Volume Control/Buffered_DAC_HP_R -> /Volume Control/DAC_CTRL_2_R
- U17 pad 5: -15V -> Net-(R67-Pad1)
- U17 pad 7: -15V -> +15V
- U21 pad 1: Net-(R103-Pad1) -> Net-(C73-Pad1)
- U21 pad 2: Net-(R103-Pad2) -> Net-(R104-Pad2)
- U21 pad 3: Net-(R104-Pad2) -> Net-(R103-Pad2)
- U21 pad 5: Net-(R114-Pad1) -> Net-(R113-Pad1)
- U21 pad 6: Net-(R113-Pad1) -> Net-(R114-Pad1)
- U21 pad 7: Net-(R119-Pad1) -> Net-(C74-Pad1)
- U6 pad 11: /input selector/CS -> Net-(U6-Pad11)
- U6 pad 12: /input selector/CLK -> /MCU/IO_SCL
- U6 pad 13: /input selector/MOSI -> /MCU/IO_SDA
Routing:
- net /MCU/SCL: track 0.00 -> 83.5 mm
- net /MCU/SDA: track 0.00 -> 42.8 mm
- net /MCU/~I2C_RST: track 0.00 -> 9.59 mm
- net GND: track 0.00 -> 9.54 mm
- net +5V: track 0.00 -> 8.90 mm
