File: preamp-layout/preamp-kicad/preamp.kicad_pcb (KiCad board)
At the start: 2 copper layers, 431 parts, among them J1 Screw_Terminal_01x03, J10 Conn_01x03_Male, J11 Conn_01x02_Male, J12 Conn_01x02_Male, J13 Conn_01x02_Male, J14 Screw_Terminal_01x03, J15 Conn_01x02_Male, J16 Conn_01x02_Male, J17 Conn_01x02_Female, J18 Conn_01x02_Female, J19 Conn_01x05_Female, J2 Conn_01x02_Female, J20 Conn_01x03_Male, J26 Conn_01x03_Female, J27 Conn_01x03_Female, J28 Conn_01x03_Female, J29 Conn_01x03_Female, J3 Conn_01x02_Female, J30 Conn_01x03_Female, J31 Conn_01x03_Male, J32 Conn_01x03_Male, J35 Conn_01x03_Male, J36 Conn_01x03_Male, J37 Conn_01x03_Male, J38 Conn_01x03_Male, J39 Conn_01x03_Male, J4 Conn_01x02_Male, J40 Conn_01x03_Male, J41 Conn_01x03_Male, J42 Conn_01x03_Female, J43 Conn_01x03_Female, J44 Conn_01x02_Female, J45 Conn_01x07_Female, J46 Conn_01x07_Female, J47 Conn_01x02_Male, J48 Conn_01x02_Male, J49 Conn_01x03_Female, J5 Screw_Terminal_01x03, J50 Conn_01x03_Male, J51 Conn_01x02_Male, J52 Conn_01x03_Female, J53 Conn_01x03_Female, J54 Conn_01x03_Male, J55 Conn_01x02_Male, J56 Conn_01x03_Male, J57 Conn_01x02_Male, J58 Conn_01x03_Male, J59 Conn_01x04_Male, J6 Screw_Terminal_01x03, J60 Conn_01x04_Female, J61 Conn_01x03_Male, J62 Conn_01x03_Male, J64 Conn_01x04_Female, J65 Conn_01x04_Male, J66 Conn_01x03_Male, J67 Conn_01x03_Male, J68 Conn_01x03_Female, J69 Conn_01x03_Male, J7 Screw_Terminal_01x03, J70 XLR3, J71 XLR3, J72 XLR3, J73 XLR3, J74 Conn_01x03_Female, J75 Conn_01x03_Female, J76 Conn_01x03_Female, J77 Conn_01x03_Female, J78 Conn_01x03_Female, J79 Conn_01x03_Female, J8 Conn_01x03_Male, J80 Conn_01x03_Female, J81 Conn_01x03_Female, J82 Conn_01x02_Male, J83 Conn_01x02_Male, J84 Conn_01x05_Female, J9 Conn_01x03_Male, K2 G6JU, K3 G6JU, K4 G6JU, K5 G6JU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

Commit message: Periodic backup
Extensive changes as a result of PCB layout phase.
Parts:
- removed J39, J40, J41: Conn_01x03_Male, Connector_PinHeader_2.54mm:PinHeader_1x03_P2.54mm_Vertical
- removed J45, J46: Conn_01x07_Female, Connector_PinHeader_2.54mm:PinHeader_1x07_P2.54mm_Vertical
- removed J53: Conn_01x03_Female, Connector_PinHeader_2.54mm:PinHeader_1x03_P2.54mm_Vertical
- removed J59, J65: Conn_01x04_Male, Connector_PinHeader_2.54mm:PinHeader_1x04_P2.54mm_Vertical
- removed J60, J64: Conn_01x04_Female, Connector_PinHeader_2.54mm:PinHeader_1x04_P2.54mm_Vertical
- removed K3, K4, K5, K6: G6JU, preamp:Relay_DPDT_Omron_G6JU-2P-Y
- removed RV4: 500R, Connector_PinHeader_2.54mm:PinHeader_1x03_P2.54mm_Vertical
- removed SW10: SW_DPDT_x2, Connector_PinHeader_2.54mm:PinHeader_1x03_P2.54mm_Vertical
- added C123: 0.1uF, Capacitor_SMD:C_0805_2012Metric_Pad1.15x1.40mm_HandSolder, F.Cu at (57.6, 84.8)
- added C92: 0.1uF, Capacitor_SMD:C_0805_2012Metric_Pad1.15x1.40mm_HandSolder, F.Cu at (46.7, 71.1)
- added C93: 0.1uF, Capacitor_SMD:C_0805_2012Metric_Pad1.15x1.40mm_HandSolder, B.Cu at (46.7, 77.8)
- added D61: GREEN, LED_SMD:LED_1206_3216Metric_Pad1.42x1.75mm_HandSolder, F.Cu at (19.0, 78.0)
- added D62: GREEN, LED_SMD:LED_1206_3216Metric_Pad1.42x1.75mm_HandSolder, F.Cu at (18.9, 80.7)
- added J95: Conn_01x03_Male, Connector_JST:JST_EH_S3B-EH_1x03_P2.50mm_Horizontal, F.Cu at (12.4, 81.0)
- added J96: Conn_01x03_Male, Connector_JST:JST_EH_S3B-EH_1x03_P2.50mm_Horizontal, F.Cu at (12.4, 69.9)
- added R139: 100R, Resistor_SMD:R_1206_3216Metric_Pad1.42x1.75mm_HandSolder, F.Cu at (25.7, 64.7)
- added R140: 100R, Resistor_SMD:R_1206_3216Metric_Pad1.42x1.75mm_HandSolder, F.Cu at (19.4, 64.7)
- added R141: 100R, Resistor_SMD:R_1206_3216Metric_Pad1.42x1.75mm_HandSolder, B.Cu at (41.4, 64.7)
- added R142: 100R, Resistor_SMD:R_1206_3216Metric_Pad1.42x1.75mm_HandSolder, B.Cu at (35.1, 64.7)
- added R143: 100R, Resistor_SMD:R_1206_3216Metric_Pad1.42x1.75mm_HandSolder, B.Cu at (28.8, 64.7)
- added R144: 100R, Resistor_SMD:R_1206_3216Metric_Pad1.42x1.75mm_HandSolder, B.Cu at (22.5, 64.7)
- added R145: 100R, Resistor_SMD:R_1206_3216Metric_Pad1.42x1.75mm_HandSolder, B.Cu at (38.3, 64.7)
- added R146: 100R, Resistor_SMD:R_1206_3216Metric_Pad1.42x1.75mm_HandSolder, B.Cu at (32.0, 64.7)
- added R147: 100R, Resistor_SMD:R_1206_3216Metric_Pad1.42x1.75mm_HandSolder, B.Cu at (25.7, 64.7)
- added R148: 100R, Resistor_SMD:R_1206_3216Metric_Pad1.42x1.75mm_HandSolder, B.Cu at (19.4, 64.7)
- added REF**: MountingHole_3.2mm_M3_DIN965, MountingHole:MountingHole_3.2mm_M3_DIN965, F.Cu at (305.2, 328.8)
- added REF**: MountingHole_3.2mm_M3_DIN965, MountingHole:MountingHole_3.2mm_M3_DIN965, F.Cu at (305.2, 370.0)
- added REF**: MountingHole_3.2mm_M3_DIN965, MountingHole:MountingHole_3.2mm_M3_DIN965, F.Cu at (217.2, 370.5)
- added REF**: MountingHole_3.2mm_M3_DIN965, MountingHole:MountingHole_3.2mm_M3_DIN965, F.Cu at (217.0, 328.2)
- added REF**: MountingHole_3.2mm_M3_DIN965, MountingHole:MountingHole_3.2mm_M3_DIN965, F.Cu at (319.8, 290.2)
- added REF**: MountingHole_3.2mm_M3_DIN965, MountingHole:MountingHole_3.2mm_M3_DIN965, F.Cu at (319.0, 224.2)
- added REF**: MountingHole_3.2mm_M3_DIN965, MountingHole:MountingHole_3.2mm_M3_DIN965, F.Cu at (201.2, 222.8)
- added REF**: MountingHole_3.2mm_M3_DIN965, MountingHole:MountingHole_3.2mm_M3_DIN965, F.Cu at (202.5, 289.8)
- added T1: Transformer_1P_2S, preamp:164J28, F.Cu at (240.4, 256.0)
- added T2: Transformer_1P_2S, preamp:164F12, F.Cu at (248.2, 349.8)
- added U24: ULN2003, Package_SO:SOIC-16_3.9x9.9mm_P1.27mm, F.Cu at (64.4, 85.0)
- C101, C20, C94, C95, C98, C99, J56, R20, R21, R22, R23, R26, R27, R34, R36, R80, R81, R86, U11: moved to B.Cu
- C96, C97: value 0.1uF -> 100uF; footprint Capacitor_SMD:C_0805_2012Metric_Pad1.15x1.40mm_HandSolder -> Capacitor_SMD:CP_Elec_8x6.2
- J15, J16, J47, J48, J51, J55, J57: footprint Connector_JST:JST_EH_B2B-EH-A_1x02_P2.50mm_Vertical -> Connector_JST:JST_EH_S2B-EH_1x02_P2.50mm_Horizontal
- J26: value Conn_01x03_Female -> Conn_01x18_Male; footprint Connector_PinHeader_2.54mm:PinHeader_1x03_P2.54mm_Vertical -> Connector_PinHeader_2.54mm:PinHeader_1x18_P2.54mm_Vertical; moved to B.Cu
- J27: value Conn_01x03_Female -> Conn_01x08_Male; footprint Connector_PinHeader_2.54mm:PinHeader_1x03_P2.54mm_Vertical -> Connector_PinHeader_2.54mm:PinHeader_1x08_P2.54mm_Vertical; moved to B.Cu
- J28: value Conn_01x03_Female -> Conn_01x18_Female; footprint Connector_PinHeader_2.54mm:PinHeader_1x03_P2.54mm_Vertical -> Connector_PinSocket_2.54mm:PinSocket_1x18_P2.54mm_Vertical
- J29: value Conn_01x03_Female -> Conn_01x08_Female; footprint Connector_PinHeader_2.54mm:PinHeader_1x03_P2.54mm_Vertical -> Connector_PinSocket_2.54mm:PinSocket_1x08_P2.54mm_Vertical
- J30: value Conn_01x03_Female -> Conn_01x04_Female; footprint Connector_PinHeader_2.54mm:PinHeader_1x03_P2.54mm_Vertical -> Connector_PinSocket_2.54mm:PinSocket_1x04_P2.54mm_Vertical
- J31: value Conn_01x03_Male -> Conn_01x04_Male; footprint Connector_PinHeader_2.54mm:PinHeader_1x03_P2.54mm_Vertical -> Connector_PinHeader_2.54mm:PinHeader_1x04_P2.54mm_Vertical; moved to B.Cu
- J32, J38, J58: footprint Connector_PinHeader_2.54mm:PinHeader_1x03_P2.54mm_Vertical -> Connector_JST:JST_EH_B3B-EH-A_1x03_P2.50mm_Vertical
- J35: value Conn_01x03_Male -> Conn_01x05_Male; footprint Connector_PinHeader_2.54mm:PinHeader_1x03_P2.54mm_Vertical -> Connector_PinHeader_2.54mm:PinHeader_1x05_P2.54mm_Vertical
- J36: value Conn_01x03_Male -> Conn_01x05_Female; footprint Connector_PinHeader_2.54mm:PinHeader_1x03_P2.54mm_Vertical -> Connector_PinSocket_2.54mm:PinSocket_1x05_P2.54mm_Vertical; moved to B.Cu
- J37: value Conn_01x03_Male -> Conn_01x08_Male; footprint Connector_PinHeader_2.54mm:PinHeader_1x03_P2.54mm_Vertical -> Connector_JST:JST_EH_B8B-EH-A_1x08_P2.50mm_Vertical
- J4: footprint Connector_JST:JST_EH_B2B-EH-A_1x02_P2.50mm_Vertical -> Connector_PinHeader_2.54mm:PinHeader_1x02_P2.54mm_Vertical
- J42, J43: footprint Connector_PinHeader_2.54mm:PinHeader_1x03_P2.54mm_Vertical -> Connector_PinSocket_2.54mm:PinSocket_1x03_P2.54mm_Vertical
- J44: footprint Connector_PinHeader_2.54mm:PinHeader_1x02_P2.54mm_Vertical -> Connector_JST:JST_EH_S2B-EH_1x02_P2.50mm_Horizontal
- J50, J54, J61, J62: footprint Connector_JST:JST_EH_B3B-EH-A_1x03_P2.50mm_Vertical -> Connector_JST:JST_EH_S3B-EH_1x03_P2.50mm_Horizontal
- J52: value Conn_01x03_Female -> Conn_01x03_Male; moved to B.Cu
- R24, R25: value 51R -> 1.5k
- R28, R29, R30, R31, R32, R33: value 51R -> 100R
- U10: value ULN2003 -> DG408DY
- U9: value ULN2003 -> DG408DY; moved to B.Cu
- moved J50 472.9 mm to (109.5, 39.4)
- moved J43 472.3 mm to (28.2, 94.8), turned to 0 degrees
- moved R35 458.8 mm to (114.0, 34.5), turned to 270 degrees
- moved J54 455.3 mm to (109.5, 50.5)
- moved R31 451.9 mm to (22.5, 64.7)
- moved R33 451.4 mm to (32.0, 64.7)
- moved D53 450.8 mm to (114.0, 40.0), turned to 90 degrees
- moved R22 446.9 mm to (63.8, 88.8)
- moved K8 446.2 mm to (62.2, 93.8)
- moved R23 445.3 mm to (60.6, 88.8)
- moved D54 443.4 mm to (114.0, 45.5), turned to 90 degrees
- moved R37 443.2 mm to (114.0, 51.0), turned to 90 degrees
- moved R30 441.2 mm to (28.8, 64.7)
- moved R32 440.9 mm to (38.3, 64.7)
- moved J55 435.6 mm to (109.5, 58.7)
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Connections:
- C101 pad 2: Net-(C101-Pad2) -> /headphone amp/Headphone Crossfeed/SW_R_OUT_1
- C19 pad 1: +5V -> +15V
- C20 pad 1: +5V -> +15V
- C98 pad 2: Net-(C98-Pad2) -> /headphone amp/Headphone Crossfeed/SW_L_OUT_1
- J26 pad 1: /IO/A_IN_1_L -> GND
- J26 pad 2: GND -> /IO/A_IN_1_L
- J27 pad 1: /IO/A_IN_2_L -> GND
- J27 pad 2: GND -> /IO/A_OUT_1_L
- J27 pad 3: /IO/A_IN_2_R -> /IO/A_OUT_1_R
- J28 pad 1: /IO/A_IN_3_L -> GND
- J28 pad 2: GND -> /IO/A_IN_1_L
- J28 pad 3: /IO/A_IN_3_R -> /IO/A_IN_1_R
- J29 pad 1: /IO/A_IN_4_L -> GND
- J29 pad 2: GND -> /IO/A_OUT_1_L
- J29 pad 3: /IO/A_IN_4_R -> /IO/A_OUT_1_R
- J30 pad 1: /IO/A_IN_5_L -> +15V
- J30 pad 2: GND -> -15V
- J30 pad 3: /IO/A_IN_5_R -> +5V
- J31 pad 1: /IO/A_OUT_1_L -> +15V
- J31 pad 2: GND -> -15V
- J31 pad 3: /IO/A_OUT_1_R -> +5V
- J32 pad 1: /IO/A_OUT_2_L -> /headphone amp/OUT_L
- J32 pad 2: GND -> /headphone amp/OUT_R
- J32 pad 3: /IO/A_OUT_2_R -> GND
- J35 pad 1: /IO/A_IN_1_L -> /headphone amp/IN_L
- J35 pad 2: GND -> /headphone amp/xfeed_out_l
- J35 pad 3: /IO/A_IN_1_R -> /headphone amp/IN_R
- J36 pad 1: /IO/A_IN_2_L -> /headphone amp/IN_L
- J36 pad 2: GND -> /headphone amp/xfeed_out_l
- J36 pad 3: /IO/A_IN_2_R -> /headphone amp/IN_R
- J37 pad 1: /IO/A_IN_3_L -> /headphone amp/IN_L
- J37 pad 2: GND -> /headphone amp/Headphone Crossfeed/VR_L_OUT
- J37 pad 3: /IO/A_IN_3_R -> /headphone amp/Headphone Crossfeed/SW_L_OUT_1
- J38 pad 1: /IO/A_IN_4_L -> /headphone amp/IN_L
- J38 pad 3: /IO/A_IN_4_R -> /headphone amp/IN_R
- K2 pad 1: /input selector/IN_1_S+ -> /input selector/OUT_3_S+
- K2 pad 2: Net-(K2-Pad2) -> GND
- K2 pad 3: /IO/A_IN_1_L -> /input selector/A_OUT_3_L
- K2 pad 4: /input selector/A_OUT_L -> /input selector/A_IN_L
- K2 pad 5: /input selector/A_OUT_R -> /input selector/A_IN_R
- K2 pad 6: /IO/A_IN_1_R -> /input selector/A_OUT_3_R
- K2 pad 7: Net-(K2-Pad7) -> GND
- K2 pad 8: /input selector/IN_1_R+ -> /input selector/OUT_3_R+
- R24 pad 1: +5V -> +15V
- R24 pad 2: /input selector/IN_1_S+ -> Net-(D61-Pad2)
- R25 pad 1: +5V -> -15V
- R25 pad 2: /input selector/IN_1_R+ -> Net-(D62-Pad1)
- R26 pad 2: /input selector/IN_2_S+ -> /input selector/OUT_3_S+
- R27 pad 2: /input selector/IN_2_R+ -> /input selector/OUT_3_R+
- R28 pad 1: +5V -> Net-(R28-Pad1)
- R28 pad 2: /input selector/IN_3_S+ -> /IO/A_IN_1_L
- R29 pad 1: +5V -> Net-(R29-Pad1)
- R29 pad 2: /input selector/IN_3_R+ -> /IO/A_IN_2_L
- R30 pad 1: +5V -> Net-(R30-Pad1)
- R30 pad 2: /input selector/IN_4_S+ -> /IO/A_IN_3_L
- R31 pad 1: +5V -> Net-(R31-Pad1)
- R31 pad 2: /input selector/IN_4_R+ -> /IO/A_IN_4_L
- R32 pad 1: +5V -> Net-(R32-Pad1)
- R32 pad 2: /input selector/IN_5_S+ -> /IO/A_IN_5_L
- R33 pad 1: +5V -> Net-(R33-Pad1)
- R33 pad 2: /input selector/IN_5_R+ -> /input selector/A_IN_6_L
- R77 pad 1: Net-(R77-Pad1) -> /headphone amp/Headphone Crossfeed/VR_L_OUT
- R79 pad 1: Net-(C98-Pad2) -> /headphone amp/Headphone Crossfeed/SW_L_OUT_1
- R80 pad 1: Net-(R80-Pad1) -> /headphone amp/Headphone Crossfeed/SW_L_OUT_2
- R83 pad 1: Net-(R83-Pad1) -> /headphone amp/Headphone Crossfeed/SW_R_OUT_2
- R84 pad 1: Net-(C101-Pad2) -> /headphone amp/Headphone Crossfeed/SW_R_OUT_1
- R85 pad 1: Net-(R85-Pad1) -> /headphone amp/Headphone Crossfeed/VR_R_OUT
- U10 pad 1: Net-(J46-Pad1) -> /input selector/IN_L_SEL_A0
- U10 pad 10: /input selector/OUT_2_R+ -> Net-(R139-Pad1)
- U10 pad 11: /input selector/OUT_2_S+ -> Net-(R33-Pad1)
- U10 pad 12: /input selector/OUT_1_R+ -> Net-(R32-Pad1)
- U10 pad 13: /input selector/OUT_1_S+ -> +15V
- U10 pad 14: /input selector/IN_5_R+ -> GND
- U10 pad 15: /input selector/IN_5_S+ -> /input selector/IN_L_SEL_A2
- U10 pad 16: /input selector/IN_4_R+ -> /input selector/IN_L_SEL_A1
- U10 pad 2: Net-(J46-Pad2) -> +15V
- U10 pad 3: Net-(J46-Pad3) -> -15V
- U10 pad 4: Net-(J46-Pad4) -> Net-(R28-Pad1)
- U10 pad 5: Net-(J46-Pad5) -> Net-(R29-Pad1)
- U10 pad 6: Net-(J46-Pad6) -> Net-(R30-Pad1)
- U10 pad 7: Net-(J46-Pad7) -> Net-(R31-Pad1)
- U10 pad 8: GND -> /input selector/A_OUT_L
- U10 pad 9: +5V -> Net-(R140-Pad1)
- U8 pad 1: Net-(J45-Pad1) -> /input selector/IN_L_SEL_A0
- U8 pad 2: Net-(J45-Pad2) -> /input selector/IN_L_SEL_A1
- U8 pad 21: Net-(J46-Pad1) -> Net-(U8-Pad21)
- U8 pad 22: Net-(J46-Pad2) -> Net-(U8-Pad22)
- U8 pad 23: Net-(J46-Pad3) -> Net-(U8-Pad23)
- U8 pad 24: Net-(J46-Pad4) -> Net-(U8-Pad24)
- U8 pad 25: Net-(J46-Pad5) -> Net-(U24-Pad1)
- U8 pad 26: Net-(J46-Pad6) -> Net-(U24-Pad2)
- U8 pad 27: Net-(J46-Pad7) -> Net-(U24-Pad3)
- U8 pad 3: Net-(J45-Pad3) -> /input selector/IN_L_SEL_A2
- U8 pad 4: Net-(J45-Pad4) -> /input selector/IN_R_SEL_A0
- U8 pad 5: Net-(J45-Pad5) -> /input selector/IN_R_SEL_A1
- U8 pad 6: Net-(J45-Pad6) -> /input selector/IN_R_SEL_A2
- U8 pad 7: Net-(J45-Pad7) -> Net-(U8-Pad7)
- U9 pad 1: Net-(J45-Pad1) -> /input selector/IN_R_SEL_A0
- U9 pad 10: /input selector/IN_4_S+ -> Net-(R147-Pad1)
- U9 pad 11: /input selector/IN_3_R+ -> Net-(R146-Pad1)
- U9 pad 12: /input selector/IN_3_S+ -> Net-(R145-Pad1)
- U9 pad 13: /input selector/IN_2_R+ -> +15V
- U9 pad 14: /input selector/IN_2_S+ -> GND
- U9 pad 15: /input selector/IN_1_R+ -> /input selector/IN_R_SEL_A2
- U9 pad 16: /input selector/IN_1_S+ -> /input selector/IN_R_SEL_A1
- U9 pad 2: Net-(J45-Pad2) -> +15V
- U9 pad 3: Net-(J45-Pad3) -> -15V
- U9 pad 4: Net-(J45-Pad4) -> Net-(R141-Pad1)
- U9 pad 5: Net-(J45-Pad5) -> Net-(R142-Pad1)
- U9 pad 6: Net-(J45-Pad6) -> Net-(R143-Pad1)
- U9 pad 7: Net-(J45-Pad7) -> Net-(R144-Pad1)
- U9 pad 8: GND -> /input selector/A_OUT_R
- U9 pad 9: +5V -> Net-(R148-Pad1)
Routing:
- net -15V: track 104.2 -> 370.7 mm, vias 0 -> 5
- net +15V: track 109.1 -> 352.9 mm, vias 0 -> 3
- net +5V: track 0.00 -> 113.4 mm
- net GND: track 132.0 -> 233.1 mm, vias 0 -> 26
- net /Volume Control/DAC_CTRL_2_R: track 0.00 -> 91.0 mm, vias 0 -> 2
- net /input selector/A_OUT_L: track 0.00 -> 75.9 mm
- net /input selector/A_OUT_R: track 0.00 -> 73.7 mm
- net /Volume Control/DAC_CTRL_2_L: track 0.00 -> 65.4 mm, vias 0 -> 2
- net /+-15V PWR SUPPLY/AC_N: track 0.00 -> 61.5 mm
- net /Volume Control/DAC_CTRL_1_R: track 0.00 -> 58.2 mm, vias 0 -> 2
- net /Volume Control/DAC_CTRL_1_L: track 0.00 -> 50.7 mm, vias 0 -> 2
- net /headphone amp/IN_R: track 22.5 -> 63.8 mm
- net Net-(C14-Pad2): track 0.00 -> 40.6 mm
- net /Volume Control/DAC_D: track 0.00 -> 37.6 mm, vias 0 -> 1
- net /Volume Control/DAC_A: track 0.00 -> 37.1 mm, vias 0 -> 1
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- added copper zone on B.Cu, net GND
Other:
- board outline added: 359.4 x 351.2 mm
- net class 15v_pwr added: clearance 0.2, trace_width 0.25, via_dia 0.8, via_drill 0.4
- net class 3.3v_pwr added: clearance 0.2, trace_width 0.25, via_dia 0.8, via_drill 0.4
- net class 5v_pwr added: clearance 0.2, trace_width 0.25, via_dia 0.8, via_drill 0.4
- net class ac_pwr added: clearance 1, trace_width 2, via_dia 0.8, via_drill 0.4
- net class analog_signal added: clearance 0.2, trace_width 0.25, via_dia 0.8, via_drill 0.4
- net class digital_signal added: clearance 0.2, trace_width 0.25, via_dia 0.8, via_drill 0.4

Commit message: PCB layout
trying a different layout for the gain stage board, this serves as a reference point.
Parts:
- removed J31: Conn_01x04_Male, Connector_PinHeader_2.54mm:PinHeader_1x04_P2.54mm_Vertical
- removed REF** (x8): MountingHole_3.2mm_M3_DIN965, MountingHole:MountingHole_3.2mm_M3_DIN965
- C123, C19, C20, C21, C72, C73, C76, C77, C78, C79, C82, C83, C84, C85, C92, C93, C94, C95: footprint Capacitor_SMD:C_0805_2012Metric_Pad1.15x1.40mm_HandSolder -> Capacitor_SMD:C_1206_3216Metric_Pad1.42x1.75mm_HandSolder
- C74, C75, C90, C91, R59, R60, R65, R66, U13, U16: moved to B.Cu
- C86, C87, C88, C89: footprint Capacitor_SMD:C_0805_2012Metric_Pad1.15x1.40mm_HandSolder -> Capacitor_SMD:C_1206_3216Metric_Pad1.42x1.75mm_HandSolder; moved to B.Cu
- moved C89 11.0 mm to (180.5, 69.2)
- moved C87 10.8 mm to (180.8, 43.2)
- moved J50 8.87 mm to (118.0, 37.0)
- moved D53 8.86 mm to (122.5, 37.5)
- moved D54 8.86 mm to (122.5, 43.0)
- moved R35 8.86 mm to (122.5, 32.0)
- moved R37 8.86 mm to (122.5, 48.5)
- moved U11 8.80 mm to (127.8, 52.0)
- moved J54 8.78 mm to (118.0, 48.5)
- moved J55 8.64 mm to (118.0, 57.4)
- moved J57 8.57 mm to (118.0, 66.4)
- moved D55 8.56 mm to (122.5, 57.8)
- moved R38 8.56 mm to (122.5, 63.8)
- moved J51 8.55 mm to (118.0, 75.4)
- moved R34 8.50 mm to (122.8, 75.8)
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Connections:
- R24 pad 1: +15V -> Net-(D61-Pad2)
- R24 pad 2: Net-(D61-Pad2) -> +15V
- U11 pad 1: /Volume Control/DAC_A -> /Volume Control/DAC_B
- U11 pad 2: /Volume Control/DAC_B -> /Volume Control/DAC_A
- U11 pad 4: /Volume Control/DAC_C -> /Volume Control/DAC_D
- U11 pad 5: /Volume Control/DAC_D -> /Volume Control/DAC_C
- U14 pad 2: /Volume Control/DAC_CTRL_1_L -> /Volume Control/DAC_CTRL_2_L
- U15 pad 2: /Volume Control/DAC_CTRL_1_R -> /Volume Control/DAC_CTRL_2_R
- U17 pad 2: /Volume Control/DAC_CTRL_2_L -> /Volume Control/DAC_CTRL_1_L
- U18 pad 2: /Volume Control/DAC_CTRL_2_R -> /Volume Control/DAC_CTRL_1_R
Routing:
- net -15V: track 370.7 -> 172.6 mm, vias 5 -> 4
- net +15V: track 352.9 -> 159.2 mm, vias 3 -> 5
- net +5V: track 113.4 -> 21.1 mm
- net GND: track 233.1 -> 147.8 mm, vias 26 -> 16
- net /+-15V PWR SUPPLY/AC_N: track 61.5 -> 0.00 mm
- net /headphone amp/IN_L: track 69.1 -> 13.2 mm
- net /Volume Control/DAC_CTRL_2_R: track 91.0 -> 37.0 mm
- net /headphone amp/IN_R: track 63.8 -> 14.4 mm
- net Net-(C14-Pad2): track 40.6 -> 0.00 mm
- net /+-15V PWR SUPPLY/rectified_+: track 39.5 -> 0.00 mm
- net Net-(F3-Pad1): track 36.7 -> 0.00 mm
- net /+-15V PWR SUPPLY/AC_HOT: track 35.5 -> 0.00 mm
- net /+-15V PWR SUPPLY/rectified_-: track 35.2 -> 0.00 mm
- net /headphone amp/OUT_L: track 34.1 -> 0.00 mm
- net Net-(C5-Pad2): track 28.8 -> 0.00 mm
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- removed copper zone on B.Cu, net GND
Other:
- outline, holes or cut-outs redrawn
- net class 15v_pwr: clearance 0.2 -> 0.4; trace_width 0.25 -> 0.5
- net class 3.3v_pwr: clearance 0.2 -> 0.4; trace_width 0.25 -> 0.5
