File: preamp-layout/preamp-kicad/preamp.kicad_pcb (KiCad board)
At the start: 2 copper layers, 359.4 x 351.2 mm, 430 parts, among them J1 Screw_Terminal_01x03, J10 Conn_01x03_Male, J11 Conn_01x02_Male, J12 Conn_01x02_Male, J13 Conn_01x02_Male, J14 Screw_Terminal_01x03, J15 Conn_01x02_Male, J16 Conn_01x02_Male, J17 Conn_01x02_Female, J18 Conn_01x02_Female, J19 Conn_01x05_Female, J2 Conn_01x02_Female, J20 Conn_01x03_Male, J26 Conn_01x18_Male, J27 Conn_01x08_Male, J28 Conn_01x18_Female, J29 Conn_01x08_Female, J3 Conn_01x02_Female, J30 Conn_01x04_Female, J32 Conn_01x03_Male, J35 Conn_01x05_Male, J36 Conn_01x05_Female, J37 Conn_01x08_Male, J38 Conn_01x03_Male, J4 Conn_01x02_Male, J42 Conn_01x03_Female, J43 Conn_01x03_Female, J44 Conn_01x02_Female, J47 Conn_01x02_Male, J48 Conn_01x02_Male, J49 Conn_01x03_Female, J5 Screw_Terminal_01x03, J50 Conn_01x03_Male, J51 Conn_01x02_Male, J52 Conn_01x03_Male, J54 Conn_01x03_Male, J55 Conn_01x02_Male, J56 Conn_01x03_Male, J57 Conn_01x02_Male, J58 Conn_01x03_Male, J6 Screw_Terminal_01x03, J61 Conn_01x03_Male, J62 Conn_01x03_Male, J66 Conn_01x03_Male, J67 Conn_01x03_Male, J68 Conn_01x03_Female, J69 Conn_01x03_Male, J7 Screw_Terminal_01x03, J70 XLR3, J71 XLR3, J72 XLR3, J73 XLR3, J74 Conn_01x03_Female, J75 Conn_01x03_Female, J76 Conn_01x03_Female, J77 Conn_01x03_Female, J78 Conn_01x03_Female, J79 Conn_01x03_Female, J8 Conn_01x03_Male, J80 Conn_01x03_Female, J81 Conn_01x03_Female, J82 Conn_01x02_Male, J83 Conn_01x02_Male, J84 Conn_01x05_Female, J9 Conn_01x03_Male, J95 Conn_01x03_Male, J96 Conn_01x03_Male, K2 G6JU, K7 G6JU, K8 G6JU, T1 Transformer_1P_2S, T2 Transformer_1P_2S, U1 LM7815, U10 DG408DY, U11 DAC5574, U12 TL074CDR, U13 NJM2068M, U14 THAT2181, U15 THAT2181, U16 NJM2068M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

Commit message: PCB layout
Parts:
- removed C10, C11, C16: 100uF, Capacitor_THT:CP_Radial_D6.3mm_P2.50mm
- removed C12, C13, C4, C5: 2200uF, Capacitor_THT:CP_Radial_D12.5mm_P5.00mm
- removed C14, C15, C6, C7, C8, C9: 0.1uF, Capacitor_SMD:C_0805_2012Metric_Pad1.15x1.40mm_HandSolder
- removed D1, D10: DF02M, Diode_THT:Diode_Bridge_DIP-4_W7.62mm_P5.08mm
- removed D11, D4, D5, D6, D7, D9: SM4001, Diode_SMD:D_SOD-123F
- removed J30: Conn_01x04_Female, Connector_PinSocket_2.54mm:PinSocket_1x04_P2.54mm_Vertical
- removed J57: Conn_01x02_Male, Connector_JST:JST_EH_S2B-EH_1x02_P2.50mm_Horizontal
- removed J61, J62, J95, J96: Conn_01x03_Male, Connector_JST:JST_EH_S3B-EH_1x03_P2.50mm_Horizontal
- removed J66, J69: Conn_01x03_Male, Connector_JST:JST_EH_B3B-EH-A_1x03_P2.50mm_Vertical
- removed J68: Conn_01x03_Female, Connector_PinHeader_2.54mm:PinHeader_1x03_P2.54mm_Vertical
- removed J82, J83: Conn_01x02_Male, Connector_JST:JST_EH_B2B-EH-A_1x02_P2.50mm_Vertical
- removed R101, R105, R106, R107, R110, R111, R112, R117, R118, R89, R92, R93, R94, R99: 10k, Resistor_SMD:R_1206_3216Metric_Pad1.42x1.75mm_HandSolder
- removed R113, R114, R95, R96: 9.09k, Resistor_SMD:R_1206_3216Metric_Pad1.42x1.75mm_HandSolder
- removed R139, R140, R141, R142, R143, R144, R145, R146, R147, R148: 100R, Resistor_SMD:R_1206_3216Metric_Pad1.42x1.75mm_HandSolder
- removed RV1, RV2, RV3: 4.7k, Potentiometer_THT:Potentiometer_Bourns_3386P_Vertical
- removed T1: Transformer_1P_2S, preamp:164J28
- removed T2: Transformer_1P_2S, preamp:164F12
- removed U12: TL074CDR, Package_SO:SOIC-14_3.9x8.7mm_P1.27mm
- removed U3: LM7805, Package_TO_SOT_THT:TO-220-3_Vertical
- added J31: Conn_01x04_Male, Connector_JST:JST_EH_S4B-EH_1x04_P2.50mm_Horizontal, F.Cu at (-46.2, 74.1)
- added J39: Conn_01x04_Male, Connector_JST:JST_EH_S4B-EH_1x04_P2.50mm_Horizontal, F.Cu at (-46.2, 59.6)
- added J40: Conn_01x04_Male, Connector_JST:JST_EH_S4B-EH_1x04_P2.50mm_Horizontal, F.Cu at (-37.8, 122.4)
- added J41: Conn_01x04_Male, Connector_JST:JST_EH_S4B-EH_1x04_P2.50mm_Horizontal, F.Cu at (-37.8, 107.8)
- added J53: Conn_01x04_Male, Connector_JST:JST_EH_B4B-EH-A_1x04_P2.50mm_Vertical, F.Cu at (82.3, 154.8)
- added PS1: IRM-10-15, Converter_ACDC:Converter_ACDC_MeanWell_IRM-10-xx_THT, F.Cu at (210.1, 137.5)
- added PS2: IRM-10-15, Converter_ACDC:Converter_ACDC_MeanWell_IRM-10-xx_THT, F.Cu at (210.1, 164.4)
- added PS3: IRM-05-5, Converter_ACDC:Converter_ACDC_MeanWell_IRM-05-xx_THT, F.Cu at (225.0, 210.0)
- added R55: 100R, Resistor_SMD:R_1206_3216Metric_Pad1.42x1.75mm_HandSolder, B.Cu at (-18.0, 42.4)
- added R61: 100R, Resistor_SMD:R_1206_3216Metric_Pad1.42x1.75mm_HandSolder, B.Cu at (-20.6, 42.4)
- C102, C103, C104, C105, C106, C107, C19, C92, R18, R19, R28, R29, R30, R31, R32, R33, R43, R44, R45, R46, R47, R48, R49, R50, U10: moved to B.Cu
- C108, C109, C111, C112: value 3300pF -> 470pF
- C2, C3: value 2200uF -> 0.1uF; footprint Capacitor_THT:CP_Radial_D12.5mm_P5.00mm -> Capacitor_SMD:C_1206_3216Metric_Pad1.42x1.75mm_HandSolder; moved to B.Cu
- J15, J16, J47, J48, J55: value Conn_01x02_Male -> Conn_01x04_Male; footprint Connector_JST:JST_EH_S2B-EH_1x02_P2.50mm_Horizontal -> Connector_JST:JST_EH_S4B-EH_1x04_P2.50mm_Horizontal
- J50: value Conn_01x03_Male -> Conn_01x04_Male; footprint Connector_JST:JST_EH_S3B-EH_1x03_P2.50mm_Horizontal -> Connector_JST:JST_EH_B4B-EH-A_1x04_P2.50mm_Vertical
- J54: value Conn_01x03_Male -> Conn_01x04_Male; footprint Connector_JST:JST_EH_S3B-EH_1x03_P2.50mm_Horizontal -> Connector_JST:JST_EH_S4B-EH_1x04_P2.50mm_Horizontal
- J67: value Conn_01x03_Male -> Conn_01x05_Male; footprint Connector_PinHeader_2.54mm:PinHeader_1x03_P2.54mm_Vertical -> Connector_PinHeader_2.54mm:PinHeader_1x05_P2.54mm_Vertical
- R10, R6, R7: value 240R -> 100R; moved to B.Cu
- R108, R109, R90, R91: value 909R -> 100R
- R34, R36: moved to F.Cu
- R4, R5, R9: value 10R 1W -> 100R; footprint Resistor_THT:R_Axial_DIN0414_L11.9mm_D4.5mm_P15.24mm_Horizontal -> Resistor_SMD:R_1206_3216Metric_Pad1.42x1.75mm_HandSolder; moved to B.Cu
- R71, R72: value 499R -> 1k
- R87, R88: value 10k -> 100R; moved to B.Cu
- U1: value LM7815 -> TL072; footprint Package_TO_SOT_THT:TO-220-3_Vertical -> Package_SO:SOIC-8_3.9x4.9mm_P1.27mm; moved to B.Cu
- U2: value LM7915 -> TL072; footprint Package_TO_SOT_THT:TO-220-3_Vertical -> Package_SO:SOIC-8_3.9x4.9mm_P1.27mm; moved to B.Cu
- U20: value NJM2068M -> THAT1280; footprint Package_SO:SOP-8_3.9x4.9mm_P1.27mm -> Package_SO:SOIC-14_3.9x8.7mm_P1.27mm
- U21, U22: value NJM2068M -> THAT1646; footprint Package_SO:SOP-8_3.9x4.9mm_P1.27mm -> Package_SO:SOIC-8_3.9x4.9mm_P1.27mm
- moved R10 433.2 mm to (-0.23, 42.4), turned to 90 degrees
- moved R9 410.3 mm to (2.31, 42.4), turned to 90 degrees
- moved R5 390.0 mm to (-12.9, 42.4), turned to 90 degrees
- moved U2 369.5 mm to (-18.5, 103.8)
- moved R7 369.5 mm to (-7.85, 42.4)
- moved R6 367.2 mm to (-10.4, 42.4), turned to 90 degrees
- moved R4 359.8 mm to (-15.5, 42.4), turned to 90 degrees
- moved C3 347.7 mm to (-22.5, 96.2), turned to 0 degrees
- moved U1 340.6 mm to (-18.5, 122.8)
- moved C2 318.5 mm to (-14.5, 108.5), turned to 0 degrees
- moved C22 252.7 mm to (130.2, -89.2)
- moved C23 252.7 mm to (103.4, -62.7)
- moved C24 252.7 mm to (117.0, -76.6)
- moved C25 252.7 mm to (121.7, -82.5)
- moved C26 252.7 mm to (125.4, -86.2)
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Connections:
- net /IO/A_IN_6_L renamed Net-(J28-Pad12)
- net /IO/A_IN_6_R renamed Net-(J28-Pad13)
- net /IO/A_IN_7_L renamed Net-(J28-Pad14)
- net /IO/A_IN_7_R renamed Net-(J28-Pad15)
- net /IO/A_IN_8_L renamed Net-(J28-Pad16)
- net /IO/A_IN_8_R renamed Net-(J28-Pad17)
- C2 pad 1: /+-15V PWR SUPPLY/rectified_+ -> +15V
- C3 pad 2: /+-15V PWR SUPPLY/rectified_- -> -15V
- C71 pad 1: Net-(C71-Pad1) -> /input selector/A_OUT_L
- C81 pad 1: Net-(C81-Pad1) -> /input selector/A_OUT_R
- J15 pad 1: +5V -> +15V
- J15 pad 2: GND -> -15V
- J16 pad 1: +5V -> +15V
- J16 pad 2: GND -> -15V
- J26 pad 10: /IO/A_IN_5_L -> /IO/A_IN_1_R
- J26 pad 11: /IO/A_IN_5_R -> /IO/A_IN_2_R
- J26 pad 12: /input selector/A_IN_6_L -> /IO/A_IN_3_R
- J26 pad 13: /input selector/A_IN_6_R -> /IO/A_IN_4_R
- J26 pad 14: /input selector/A_IN_7_L -> /IO/A_IN_5_R
- J26 pad 15: /input selector/A_IN_7_R -> /input selector/A_IN_6_R
- J26 pad 16: /input selector/A_IN_8_L -> /input selector/A_IN_7_R
- J26 pad 3: /IO/A_IN_1_R -> /IO/A_IN_2_L
- J26 pad 4: /IO/A_IN_2_L -> /IO/A_IN_3_L
- J26 pad 5: /IO/A_IN_2_R -> /IO/A_IN_4_L
- J26 pad 6: /IO/A_IN_3_L -> /IO/A_IN_5_L
- J26 pad 7: /IO/A_IN_3_R -> /input selector/A_IN_6_L
- J26 pad 8: /IO/A_IN_4_L -> /input selector/A_IN_7_L
- J26 pad 9: /IO/A_IN_4_R -> /input selector/A_IN_8_L
- J28 pad 10: /IO/A_IN_5_L -> Net-(J28-Pad10)
- J28 pad 11: /IO/A_IN_5_R -> Net-(J28-Pad11)
- J28 pad 2: /IO/A_IN_1_L -> Net-(J28-Pad2)
- J28 pad 3: /IO/A_IN_1_R -> Net-(J28-Pad3)
- J28 pad 4: /IO/A_IN_2_L -> Net-(J28-Pad4)
- J28 pad 5: /IO/A_IN_2_R -> Net-(J28-Pad5)
- J28 pad 6: /IO/A_IN_3_L -> Net-(J28-Pad6)
- J28 pad 7: /IO/A_IN_3_R -> Net-(J28-Pad7)
- J28 pad 8: /IO/A_IN_4_L -> Net-(J28-Pad8)
- J28 pad 9: /IO/A_IN_4_R -> Net-(J28-Pad9)
- J38 pad 2: GND -> /headphone amp/IN_R
- J38 pad 3: /headphone amp/IN_R -> GND
- J42 pad 2: GND -> /input selector/A_IN_R
- J42 pad 3: /input selector/A_IN_R -> GND
- J43 pad 2: GND -> /input selector/A_OUT_R
- J43 pad 3: /input selector/A_OUT_R -> GND
- J47 pad 1: +5V -> +15V
- J47 pad 2: GND -> -15V
- J48 pad 1: +5V -> +15V
- J48 pad 2: GND -> -15V
- J50 pad 2: GND -> -15V
- J50 pad 3: -15V -> GND
- J52 pad 2: GND -> /input selector/A_IN_R
- J52 pad 3: /input selector/A_IN_R -> GND
- J54 pad 2: GND -> -15V
- J54 pad 3: -15V -> GND
- J55 pad 1: +5V -> +15V
- J55 pad 2: GND -> -15V
- J56 pad 1: Net-(C71-Pad1) -> /input selector/A_OUT_L
- J56 pad 2: GND -> /input selector/A_OUT_R
- J56 pad 3: Net-(C81-Pad1) -> GND
- J67 pad 2: GND -> /IO/A_OUT_2_R
- J67 pad 3: /IO/A_OUT_2_R -> GND
- R10 pad 1: +5V -> Net-(R10-Pad1)
- R10 pad 2: GND -> /IO/A_IN_2_L
- R115 pad 2: Net-(R111-Pad1) -> Net-(R115-Pad2)
- R116 pad 2: Net-(R112-Pad1) -> Net-(R116-Pad2)
- R28 pad 2: /IO/A_IN_1_L -> /IO/A_IN_3_L
- R29 pad 2: /IO/A_IN_2_L -> /IO/A_IN_4_L
- R30 pad 2: /IO/A_IN_3_L -> /input selector/A_IN_8_R
- R31 pad 2: /IO/A_IN_4_L -> /input selector/A_IN_7_R
- R32 pad 2: /IO/A_IN_5_L -> /input selector/A_IN_6_R
- R33 pad 2: /input selector/A_IN_6_L -> /IO/A_IN_5_R
- R39 pad 1: Net-(C62-Pad1) -> Net-(C63-Pad1)
- R4 pad 1: Net-(C4-Pad1) -> Net-(R4-Pad1)
- R4 pad 2: /+-15V PWR SUPPLY/rectified_+ -> /input selector/A_IN_8_L
- R40 pad 1: Net-(C63-Pad1) -> Net-(C65-Pad1)
- R42 pad 1: Net-(C65-Pad1) -> Net-(C62-Pad1)
- R5 pad 1: Net-(C5-Pad2) -> Net-(R5-Pad1)
- R5 pad 2: /+-15V PWR SUPPLY/rectified_- -> /input selector/A_IN_7_L
- R56 pad 1: /input selector/A_OUT_L -> /Volume Control/A_IN_L
- R6 pad 1: +15V -> Net-(R6-Pad1)
- R6 pad 2: GND -> /input selector/A_IN_6_L
- R62 pad 1: /input selector/A_OUT_R -> /Volume Control/A_IN_R
- R7 pad 1: -15V -> Net-(R7-Pad1)
- R7 pad 2: GND -> /IO/A_IN_5_L
- R73 pad 2: Net-(R69-Pad1) -> Net-(R71-Pad1)
- R74 pad 2: Net-(R70-Pad1) -> Net-(R72-Pad1)
- R87 pad 2: /IO/A_OUT_2_L -> /IO/A_IN_3_R
- R88 pad 2: /IO/A_OUT_2_L -> /IO/A_IN_4_R
- R9 pad 1: Net-(C13-Pad1) -> Net-(R9-Pad1)
- R9 pad 2: /5V supply/rectified_+ -> /IO/A_IN_1_L
- R97 pad 2: Net-(R94-Pad1) -> Net-(R97-Pad2)
- R98 pad 2: Net-(R93-Pad1) -> Net-(R98-Pad2)
- U1 pad 1: Net-(C4-Pad1) -> /Volume Control/DAC_CTRL_2_L
- U1 pad 2: Net-(C6-Pad2) -> Net-(C66-Pad2)
- U1 pad 3: +15V -> GND
- U10 pad 10: Net-(R139-Pad1) -> Net-(R28-Pad1)
- U10 pad 11: Net-(R33-Pad1) -> Net-(R10-Pad1)
- U10 pad 12: Net-(R32-Pad1) -> Net-(R9-Pad1)
- U10 pad 4: Net-(R28-Pad1) -> Net-(R4-Pad1)
- U10 pad 5: Net-(R29-Pad1) -> Net-(R5-Pad1)
- U10 pad 6: Net-(R30-Pad1) -> Net-(R6-Pad1)
- U10 pad 7: Net-(R31-Pad1) -> Net-(R7-Pad1)
- U10 pad 9: Net-(R140-Pad1) -> Net-(R29-Pad1)
- U13 pad 1: /input selector/A_IN_L -> /input selector/A_IN_R
- U13 pad 2: Net-(C74-Pad2) -> Net-(C75-Pad2)
- U13 pad 6: Net-(C75-Pad2) -> Net-(C74-Pad2)
- U13 pad 7: /input selector/A_IN_R -> /input selector/A_IN_L
- U14 pad 1: /input selector/A_OUT_L -> /Volume Control/A_IN_L
- U15 pad 1: /input selector/A_OUT_R -> /Volume Control/A_IN_R
- U16 pad 1: /headphone amp/IN_L -> /headphone amp/IN_R
- U16 pad 2: Net-(C90-Pad2) -> Net-(C91-Pad2)
- U16 pad 6: Net-(C91-Pad2) -> Net-(C90-Pad2)
- U16 pad 7: /headphone amp/IN_R -> /headphone amp/IN_L
- U17 pad 1: /input selector/A_OUT_L -> /Volume Control/A_IN_L
- U18 pad 1: /input selector/A_OUT_R -> /Volume Control/A_IN_R
- U19 pad 16: Net-(R70-Pad1) -> Net-(R72-Pad1)
- U19 pad 17: Net-(R72-Pad1) -> Net-(R70-Pad1)
- U19 pad 4: Net-(R71-Pad1) -> Net-(R69-Pad1)
- U19 pad 5: Net-(R69-Pad1) -> Net-(R71-Pad1)
- U2 pad 1: Net-(C7-Pad2) -> /Volume Control/DAC_CTRL_1_L
- U2 pad 2: Net-(C5-Pad2) -> Net-(C68-Pad2)
- U2 pad 3: -15V -> GND
- U20 pad 1: Net-(C110-Pad1) -> (no net)
- U20 pad 2: Net-(R101-Pad2) -> Net-(C108-Pad1)
- U20 pad 3: Net-(R95-Pad1) -> Net-(C109-Pad2)
- U20 pad 5: Net-(R113-Pad1) -> Net-(C112-Pad2)
- U20 pad 6: Net-(R114-Pad1) -> Net-(C111-Pad1)
- U20 pad 7: Net-(C113-Pad1) -> (no net)
- U20 pad 8: +15V -> GND
- U21 pad 1: Net-(R94-Pad1) -> Net-(R98-Pad2)
- U21 pad 2: Net-(R92-Pad1) -> Net-(R98-Pad2)
- U21 pad 3: Net-(R87-Pad1) -> GND
- U21 pad 4: -15V -> /IO/A_OUT_2_L
- U21 pad 5: GND -> -15V
- U21 pad 6: Net-(R88-Pad1) -> +15V
- U21 pad 7: Net-(R93-Pad1) -> Net-(R97-Pad2)
- U21 pad 8: +15V -> Net-(R97-Pad2)
- U22 pad 1: Net-(R111-Pad1) -> Net-(R116-Pad2)
- U22 pad 2: Net-(R110-Pad1) -> Net-(R116-Pad2)
- U22 pad 3: Net-(R105-Pad1) -> GND
- U22 pad 4: -15V -> /IO/A_OUT_2_R
- U22 pad 5: GND -> -15V
- U22 pad 6: Net-(R106-Pad1) -> +15V
- U22 pad 7: Net-(R112-Pad1) -> Net-(R115-Pad2)
- U22 pad 8: +15V -> Net-(R115-Pad2)
- U24 pad 1: Net-(U24-Pad1) -> /input selector/RLY_1_S+
- U24 pad 2: Net-(U24-Pad2) -> /input selector/RLY_1_R+
- U24 pad 3: Net-(U24-Pad3) -> /input selector/RLY_2_S+
- U24 pad 4: Net-(U24-Pad4) -> /input selector/RLY_2_R+
- U24 pad 5: Net-(U24-Pad5) -> /input selector/RLY_3_S+
- U24 pad 6: Net-(U24-Pad6) -> /input selector/RLY_3_R+
- U8 pad 1: /input selector/IN_L_SEL_A0 -> /input selector/IN_R_SEL_A0
- U8 pad 2: /input selector/IN_L_SEL_A1 -> /input selector/IN_R_SEL_A1
- U8 pad 23: Net-(U8-Pad23) -> /input selector/RLY_3_R+
- U8 pad 24: Net-(U8-Pad24) -> /input selector/RLY_3_S+
- U8 pad 25: Net-(U24-Pad1) -> /input selector/RLY_2_R+
- U8 pad 26: Net-(U24-Pad2) -> /input selector/RLY_2_S+
- U8 pad 27: Net-(U24-Pad3) -> /input selector/RLY_1_R+
- U8 pad 28: Net-(U24-Pad4) -> /input selector/RLY_1_S+
- U8 pad 3: /input selector/IN_L_SEL_A2 -> /input selector/IN_R_SEL_A2
- U8 pad 4: /input selector/IN_R_SEL_A0 -> /input selector/IN_L_SEL_A0
- U8 pad 5: /input selector/IN_R_SEL_A1 -> /input selector/IN_L_SEL_A1
- U8 pad 6: /input selector/IN_R_SEL_A2 -> /input selector/IN_L_SEL_A2
- U9 pad 10: Net-(R147-Pad1) -> Net-(R87-Pad1)
- U9 pad 4: Net-(R141-Pad1) -> Net-(R30-Pad1)
- U9 pad 5: Net-(R142-Pad1) -> Net-(R31-Pad1)
- U9 pad 6: Net-(R143-Pad1) -> Net-(R32-Pad1)
- U9 pad 7: Net-(R144-Pad1) -> Net-(R33-Pad1)
- U9 pad 9: Net-(R148-Pad1) -> Net-(R88-Pad1)
Routing:
- net +15V: track 234.7 -> 388.0 mm, vias 4 -> 12
- net GND: track 120.3 -> 9.96 mm, vias 16 -> 11
- net +5V: track 60.3 -> 164.2 mm
- net -15V: track 316.8 -> 412.3 mm, vias 5 -> 11
- net /Volume Control/A_IN_R: track 0.00 -> 66.4 mm, vias 0 -> 4
- net /headphone amp/IN_R: track 14.4 -> 73.2 mm
- net /IO/A_IN_5_R: track 0.00 -> 53.3 mm
- net /headphone amp/IN_L: track 13.2 -> 65.6 mm
- net /Volume Control/A_IN_L: track 0.00 -> 50.9 mm, vias 0 -> 2
- net /input selector/IN_R_SEL_A0: track 0.00 -> 40.7 mm, vias 0 -> 1
- net /input selector/IN_R_SEL_A2: track 0.00 -> 38.0 mm, vias 0 -> 1
- net /input selector/IN_R_SEL_A1: track 0.00 -> 36.6 mm, vias 0 -> 1
- net /headphone amp/xfeed_out_r: track 0.00 -> 33.9 mm
- net /headphone amp/xfeed_out_l: track 0.00 -> 32.9 mm
- net /IO/A_OUT_2_R: track 0.00 -> 30.3 mm
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- added copper zone on B.Cu, net (none)
- added copper zone on F.Cu, net GND
Other:
- board size 359.4 x 351.2 mm -> 374 x 202 mm

Commit message: PCB layout update, front panel and LED restructure
Restructure of capacitive buttons. Restructure of MCU schematic. Moved LEDs to front panel sheet. Front panel and MCU initial PCB layout. 8 bit DAC update (grounded address pins). DAC connection renaming. Added mounting holes for boards.
Parts:
- removed C49, C50, C51, C52, C53, C54, C55, C56, C57, C58, C59, C60, C61: 100nF, Capacitor_SMD:C_0805_2012Metric_Pad1.15x1.40mm_HandSolder
- removed D45, D46, D47, D48, D49, D50, D51, D52: WS2812B, LED_SMD:LED_WS2812B_PLCC4_5.0x5.0mm_P3.2mm
- removed J20: Conn_01x03_Male, Connector_PinHeader_2.54mm:PinHeader_1x03_P2.54mm_Vertical
- removed J49, J74, J75, J76, J77, J78, J79, J80, J81: Conn_01x03_Female, Connector_PinHeader_2.54mm:PinHeader_1x03_P2.54mm_Vertical
- removed J54, J55: Conn_01x04_Male, Connector_JST:JST_EH_S4B-EH_1x04_P2.50mm_Horizontal
- removed U5: ESP32-DevKitC, preamp:ESP32_MELIFE_DEVKIT
- removed U6: TCA9548APWR, Package_SO:TSSOP-24_4.4x7.8mm_P0.65mm
- added C10: 100nF, Capacitor_SMD:C_0805_2012Metric_Pad1.15x1.40mm_HandSolder, F.Cu at (70.6, -32.0)
- added C11: 100nF, Capacitor_SMD:C_0805_2012Metric_Pad1.15x1.40mm_HandSolder, F.Cu at (-40.5, -32.0)
- added C12: 100nF, Capacitor_SMD:C_0805_2012Metric_Pad1.15x1.40mm_HandSolder, F.Cu at (140.0, -32.0)
- added C13: 100nF, Capacitor_SMD:C_0805_2012Metric_Pad1.15x1.40mm_HandSolder, F.Cu at (22.0, -32.0)
- added C14: 100nF, Capacitor_SMD:C_0805_2012Metric_Pad1.15x1.40mm_HandSolder, F.Cu at (195.6, -32.0)
- added C15: 100nF, Capacitor_SMD:C_0805_2012Metric_Pad1.15x1.40mm_HandSolder, F.Cu at (202.5, -32.0)
- added C16: 100nF, Capacitor_SMD:C_0805_2012Metric_Pad1.15x1.40mm_HandSolder, F.Cu at (15.0, -32.0)
- added C4: 100nF, Capacitor_SMD:C_0805_2012Metric_Pad1.15x1.40mm_HandSolder, F.Cu at (160.8, -32.0)
- added C5: 100nF, Capacitor_SMD:C_0805_2012Metric_Pad1.15x1.40mm_HandSolder, F.Cu at (153.9, -32.0)
- added C6: 100nF, Capacitor_SMD:C_0805_2012Metric_Pad1.15x1.40mm_HandSolder, F.Cu at (98.3, -32.0)
- added C7: 100nF, Capacitor_SMD:C_0805_2012Metric_Pad1.15x1.40mm_HandSolder, F.Cu at (-5.81, -32.0)
- added C8: 100nF, Capacitor_SMD:C_0805_2012Metric_Pad1.15x1.40mm_HandSolder, F.Cu at (49.7, -32.0)
- added C9: 100nF, Capacitor_SMD:C_0805_2012Metric_Pad1.15x1.40mm_HandSolder, F.Cu at (-26.6, -32.0)
- added D1: WS2812B, LED_SMD:LED_WS2812B_PLCC4_5.0x5.0mm_P3.2mm, F.Cu at (202.5, -39.0)
- added D10: WS2812B, LED_SMD:LED_WS2812B_PLCC4_5.0x5.0mm_P3.2mm, F.Cu at (105.3, -39.0)
- added D11: WS2812B, LED_SMD:LED_WS2812B_PLCC4_5.0x5.0mm_P3.2mm, F.Cu at (84.5, -39.0)
- added D4: WS2812B, LED_SMD:LED_WS2812B_PLCC4_5.0x5.0mm_P3.2mm, F.Cu at (98.3, -39.0)
- added D5: WS2812B, LED_SMD:LED_WS2812B_PLCC4_5.0x5.0mm_P3.2mm, F.Cu at (91.4, -39.0)
- added D6: WS2812B, LED_SMD:LED_WS2812B_PLCC4_5.0x5.0mm_P3.2mm, F.Cu at (-12.8, -39.0)
- added D7: WS2812B, LED_SMD:LED_WS2812B_PLCC4_5.0x5.0mm_P3.2mm, F.Cu at (-19.7, -39.0)
- added D9: WS2812B, LED_SMD:LED_WS2812B_PLCC4_5.0x5.0mm_P3.2mm, F.Cu at (195.6, -39.0)
- added H1: MountingHole, MountingHole:MountingHole_3.2mm_M3, F.Cu at (-46.0, 23.0)
- added H10: MountingHole, MountingHole:MountingHole_3.2mm_M3, F.Cu at (170.5, 119.4)
- added H11: MountingHole, MountingHole:MountingHole_3.2mm_M3, F.Cu at (178.5, 111.5)
- added H12: MountingHole, MountingHole:MountingHole_3.2mm_M3, F.Cu at (178.5, 119.4)
- added H13: MountingHole, MountingHole:MountingHole_3.2mm_M3, F.Cu at (168.5, 180.4)
- added H14: MountingHole, MountingHole:MountingHole_3.2mm_M3, F.Cu at (168.5, 172.5)
- added H15: MountingHole, MountingHole:MountingHole_3.2mm_M3, F.Cu at (160.6, 180.4)
- added H16: MountingHole, MountingHole:MountingHole_3.2mm_M3, F.Cu at (160.6, 172.5)
- added H17: MountingHole, MountingHole:MountingHole_3.2mm_M3, F.Cu at (294.0, -25.0)
- added H18: MountingHole, MountingHole:MountingHole_3.2mm_M3, F.Cu at (365.0, -25.0)
- added H19: MountingHole, MountingHole:MountingHole_3.2mm_M3, F.Cu at (294.0, 13.0)
- added H2: MountingHole, MountingHole:MountingHole_3.2mm_M3, F.Cu at (28.0, 23.0)
- added H20: MountingHole, MountingHole:MountingHole_3.2mm_M3, F.Cu at (365.0, 13.0)
- added H21: MountingHole, MountingHole:MountingHole_3.2mm_M3, F.Cu at (48.0, 23.0)
- added H22: MountingHole, MountingHole:MountingHole_3.2mm_M3, F.Cu at (104.0, 23.0)
- added H23: MountingHole, MountingHole:MountingHole_3.2mm_M3, F.Cu at (48.0, 70.0)
- added H24: MountingHole, MountingHole:MountingHole_3.2mm_M3, F.Cu at (104.0, 70.0)
- added H25: MountingHole, MountingHole:MountingHole_3.2mm_M3, F.Cu at (126.0, 26.0)
- added H26: MountingHole, MountingHole:MountingHole_3.2mm_M3, F.Cu at (162.0, 26.0)
- added H27: MountingHole, MountingHole:MountingHole_3.2mm_M3, F.Cu at (126.0, 67.0)
- added H28: MountingHole, MountingHole:MountingHole_3.2mm_M3, F.Cu at (162.0, 67.0)
- added H29: MountingHole, MountingHole:MountingHole_3.2mm_M3, F.Cu at (-13.0, 134.0)
- added H3: MountingHole, MountingHole:MountingHole_3.2mm_M3, F.Cu at (-46.0, 70.0)
- added H30: MountingHole, MountingHole:MountingHole_3.2mm_M3, F.Cu at (-13.0, 86.0)
- added H31: MountingHole, MountingHole:MountingHole_3.2mm_M3, F.Cu at (-45.0, 134.0)
- added H32: MountingHole, MountingHole:MountingHole_3.2mm_M3, F.Cu at (-45.0, 86.0)
- added H33: MountingHole, MountingHole:MountingHole_3.2mm_M3, F.Cu at (-74.0, -44.0)
- added H34: MountingHole, MountingHole:MountingHole_3.2mm_M3, F.Cu at (262.0, -44.0)
- added H35: MountingHole, MountingHole:MountingHole_3.2mm_M3, F.Cu at (-74.0, -12.0)
- added H36: MountingHole, MountingHole:MountingHole_3.2mm_M3, F.Cu at (262.0, -12.0)
- added H4: MountingHole, MountingHole:MountingHole_3.2mm_M3, F.Cu at (28.0, 70.0)
- added H5: MountingHole, MountingHole:MountingHole_3.2mm_M3, F.Cu at (21.5, 128.0)
- added H6: MountingHole, MountingHole:MountingHole_3.2mm_M3, F.Cu at (21.5, 135.9)
- added H7: MountingHole, MountingHole:MountingHole_3.2mm_M3, F.Cu at (29.4, 128.0)
- added H8: MountingHole, MountingHole:MountingHole_3.2mm_M3, F.Cu at (29.4, 135.9)
- added H9: MountingHole, MountingHole:MountingHole_3.2mm_M3, F.Cu at (170.5, 111.5)
- added J30: Conn_01x03_Female, Connector_JST:JST_EH_S3B-EH_1x03_P2.50mm_Horizontal, F.Cu at (228.0, -36.5)
- added J61: Conn_01x05_Female, Connector_PinHeader_2.54mm:PinHeader_1x05_P2.54mm_Vertical, F.Cu at (357.2, -17.2)
- added R101: 1M, Resistor_SMD:R_1206_3216Metric_Pad1.42x1.75mm_HandSolder, B.Cu at (49.7, -18.5)
- added R105: 1M, Resistor_SMD:R_1206_3216Metric_Pad1.42x1.75mm_HandSolder, B.Cu at (84.5, -18.5)
- added R106: 1M, Resistor_SMD:R_1206_3216Metric_Pad1.42x1.75mm_HandSolder, B.Cu at (119.2, -18.5)
- added R107: 1M, Resistor_SMD:R_1206_3216Metric_Pad1.42x1.75mm_HandSolder, B.Cu at (153.9, -18.5)
- added R110: 1M, Resistor_SMD:R_1206_3216Metric_Pad1.42x1.75mm_HandSolder, B.Cu at (188.6, -18.5)
- added R89: 1.5k, Resistor_SMD:R_1206_3216Metric_Pad1.42x1.75mm_HandSolder, F.Cu at (353.8, 0.91)
- added R92: 1.5k, Resistor_SMD:R_1206_3216Metric_Pad1.42x1.75mm_HandSolder, F.Cu at (353.8, -2.90)
- added R93: 1.5k, Resistor_SMD:R_1206_3216Metric_Pad1.42x1.75mm_HandSolder, F.Cu at (333.8, -6.71)
- added R94: 1.5k, Resistor_SMD:R_1206_3216Metric_Pad1.42x1.75mm_HandSolder, F.Cu at (333.8, -2.90)
- added R95: 1M, Resistor_SMD:R_1206_3216Metric_Pad1.42x1.75mm_HandSolder, B.Cu at (-54.4, -18.5)
- added R96: 1M, Resistor_SMD:R_1206_3216Metric_Pad1.42x1.75mm_HandSolder, B.Cu at (-19.7, -18.5)
- added R99: 1M, Resistor_SMD:R_1206_3216Metric_Pad1.42x1.75mm_HandSolder, B.Cu at (15.0, -18.5)
- added U3: PCA9544AD, Package_SO:SOIC-20W_7.5x12.8mm_P1.27mm, F.Cu at (344.0, -1.00)
- added U7: MCP23008T-E_SO, Package_SO:SOIC-18W_7.5x11.6mm_P1.27mm, F.Cu at (344.0, -16.9)
- C114, C115, C116, C117, C118, C119, C120, C121, C122, R121, R122, R123, R124, R125, R126, R127, R128, R133, R134, R135, U23: moved to B.Cu
- J19: value Conn_01x05_Female -> Conn_01x08_Female; footprint Connector_PinHeader_2.54mm:PinHeader_1x05_P2.54mm_Vertical -> Connector_JST:JST_EH_B8B-EH-A_1x08_P2.50mm_Vertical
- J84: value Conn_01x05_Female -> Conn_01x08_Female; footprint Connector_PinHeader_2.54mm:PinHeader_1x05_P2.54mm_Vertical -> Connector_JST:JST_EH_B8B-EH-A_1x08_P2.50mm_Vertical; moved to B.Cu
- R13: value 10k -> 1.5k
- R18, R19: moved to F.Cu
- moved C114 277.2 mm to (-54.4, -21.5)
- moved R121 263.8 mm to (-54.4, -15.5)
- moved C115 235.6 mm to (-19.7, -21.5)
- moved R122 228.6 mm to (-19.7, -15.5)
- moved C43 215.8 mm to (-68.3, -32.0), turned to 180 degrees
- moved C116 208.5 mm to (15.0, -21.5)
- moved R123 201.5 mm to (15.0, -15.5)
- moved C39 199.0 mm to (-61.4, -32.0), turned to 180 degrees
- moved D34 189.8 mm to (-54.4, -39.0), turned to 270 degrees
- moved C27 184.8 mm to (-33.6, -32.0), turned to 180 degrees
- moved C40 176.4 mm to (-54.4, -32.0)
- moved D39 175.3 mm to (-61.4, -39.0), turned to 270 degrees
- moved C29 172.0 mm to (-47.5, -32.0), turned to 180 degrees
- moved D44 164.3 mm to (-68.3, -39.0), turned to 270 degrees
- moved D19 162.0 mm to (-33.6, -39.0), turned to 270 degrees
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Connections:
- net /Volume Control/DAC_CTRL_1_L renamed /Volume Control/GAIN_CTRL_1_L
- net /Volume Control/DAC_CTRL_1_R renamed /Volume Control/GAIN_CTRL_1_R
- net /Volume Control/DAC_CTRL_2_L renamed /Volume Control/GAIN_CTRL_2_L
- net /Volume Control/DAC_CTRL_2_R renamed /Volume Control/GAIN_CTRL_2_R
- net /front panel/SW_1 renamed Net-(C114-Pad1)
- net /front panel/SW_2 renamed Net-(C115-Pad1)
- net /front panel/SW_3 renamed Net-(C116-Pad1)
- net /front panel/SW_4 renamed Net-(C117-Pad1)
- net /front panel/SW_5 renamed Net-(C118-Pad1)
- net /front panel/SW_6 renamed Net-(C119-Pad1)
- net /front panel/SW_7 renamed Net-(C120-Pad1)
- net /front panel/SW_8 renamed Net-(C121-Pad1)
- C17 pad 1: +5V -> +3.3V
- C22 pad 1: +5V -> GND
- C22 pad 2: GND -> +5V
- C23 pad 1: GND -> +5V
- C23 pad 2: +5V -> GND
- C24 pad 1: +5V -> GND
- C24 pad 2: GND -> +5V
- C25 pad 1: GND -> +5V
- C25 pad 2: +5V -> GND
- C26 pad 1: +5V -> GND
- C26 pad 2: GND -> +5V
- C27 pad 1: GND -> +5V
- C27 pad 2: +5V -> GND
- C28 pad 1: +5V -> GND
- C28 pad 2: GND -> +5V
- C29 pad 1: GND -> +5V
- C29 pad 2: +5V -> GND
- C30 pad 1: +5V -> GND
- C30 pad 2: GND -> +5V
- C31 pad 1: GND -> +5V
- C31 pad 2: +5V -> GND
- C32 pad 1: +5V -> GND
- C32 pad 2: GND -> +5V
- C33 pad 1: GND -> +5V
- C33 pad 2: +5V -> GND
- C34 pad 1: +5V -> GND
- C34 pad 2: GND -> +5V
- C35 pad 1: GND -> +5V
- C35 pad 2: +5V -> GND
- C36 pad 1: +5V -> GND
- C36 pad 2: GND -> +5V
- C37 pad 1: GND -> +5V
- C37 pad 2: +5V -> GND
- C38 pad 1: +5V -> GND
- C38 pad 2: GND -> +5V
- C39 pad 1: GND -> +5V
- C39 pad 2: +5V -> GND
- C40 pad 1: +5V -> GND
- C40 pad 2: GND -> +5V
- C41 pad 1: GND -> +5V
- C41 pad 2: +5V -> GND
- C42 pad 1: +5V -> GND
- C42 pad 2: GND -> +5V
- C43 pad 1: GND -> +5V
- C43 pad 2: +5V -> GND
- C44 pad 1: +5V -> GND
- C44 pad 2: GND -> +5V
- C45 pad 1: GND -> +5V
- C45 pad 2: +5V -> GND
- C46 pad 1: +5V -> GND
- C46 pad 2: GND -> +5V
- C47 pad 1: GND -> +5V
- C47 pad 2: +5V -> GND
- C48 pad 1: +5V -> GND
- C48 pad 2: GND -> +5V
- D13 pad 4: /MCU/LED_DT -> Net-(D13-Pad4)
- D15 pad 4: Net-(D14-Pad2) -> Net-(D15-Pad4)
- D16 pad 2: Net-(D16-Pad2) -> Net-(D10-Pad4)
- D17 pad 4: Net-(D16-Pad2) -> Net-(D11-Pad2)
- D18 pad 2: Net-(D18-Pad2) -> Net-(D13-Pad4)
- D18 pad 4: Net-(D13-Pad2) -> Net-(D18-Pad4)
- D19 pad 2: Net-(D14-Pad4) -> Net-(D19-Pad2)
- D19 pad 4: Net-(D19-Pad4) -> Net-(D14-Pad2)
- D23 pad 2: Net-(D23-Pad2) -> Net-(D18-Pad4)
- D23 pad 4: Net-(D18-Pad2) -> Net-(D23-Pad4)
- D24 pad 2: Net-(D19-Pad4) -> Net-(D24-Pad2)
- D24 pad 4: Net-(D24-Pad4) -> Net-(D19-Pad2)
- D28 pad 2: Net-(D28-Pad2) -> Net-(D23-Pad4)
- D28 pad 4: Net-(D23-Pad2) -> Net-(D28-Pad4)
- D29 pad 2: Net-(D24-Pad4) -> Net-(D29-Pad2)
- D29 pad 4: Net-(D29-Pad4) -> Net-(D24-Pad2)
- D33 pad 2: Net-(D33-Pad2) -> Net-(D28-Pad4)
- D33 pad 4: Net-(D28-Pad2) -> Net-(D33-Pad4)
- D34 pad 2: Net-(D29-Pad4) -> Net-(D34-Pad2)
- D34 pad 4: Net-(D34-Pad4) -> Net-(D29-Pad2)
- D38 pad 2: Net-(D38-Pad2) -> Net-(D33-Pad4)
- D38 pad 4: Net-(D33-Pad2) -> Net-(D38-Pad4)
- D39 pad 2: Net-(D34-Pad4) -> Net-(D39-Pad2)
- D39 pad 4: Net-(D39-Pad4) -> Net-(D34-Pad2)
- D41 pad 4: Net-(D41-Pad4) -> Net-(D40-Pad2)
- D43 pad 2: Net-(D43-Pad2) -> Net-(D38-Pad4)
- D43 pad 4: Net-(D38-Pad2) -> Net-(D42-Pad2)
- D44 pad 2: Net-(D39-Pad4) -> Net-(D44-Pad2)
- D44 pad 4: Net-(D44-Pad4) -> Net-(D39-Pad2)
- R11 pad 2: /MCU/SCL -> /MCU/SDM
- R12 pad 2: /MCU/SDA -> /MCU/SCM
- R13 pad 1: /MCU/~I2C_RST -> +3.3V
- R14 pad 2: Net-(R14-Pad2) -> /MCU/SC3
- R15 pad 2: Net-(R15-Pad2) -> /MCU/SD3
- U11 pad 10: Net-(U11-Pad10) -> GND
- U11 pad 9: Net-(U11-Pad9) -> GND
- U23 pad 19: /front panel/FP_INTA -> /MCU/ENC_INT
- U23 pad 20: /MCU/ENC_INT -> /front panel/FP_INTA
- U4 pad 13: /MCU/SDA -> /MCU/SDM
- U4 pad 14: /MCU/SCL -> /MCU/SCM
- U4 pad 6: /MCU/LED_DT -> /front panel/FP_LED_DT
- U8 pad 1: /input selector/IN_R_SEL_A0 -> /input selector/IN_R_SEL_A2
- U8 pad 3: /input selector/IN_R_SEL_A2 -> /input selector/IN_R_SEL_A0
Routing:
- net +5V: track 164.2 -> 1102.0 mm, vias 0 -> 1
- net GND: track 9.96 -> 617.1 mm, vias 11 -> 12
- net /IO/A_OUT_1_L: track 0.00 -> 103.3 mm
- net /IO/A_OUT_1_R: track 0.00 -> 92.5 mm
- net /IO/A_OUT_2_L: track 23.7 -> 111.9 mm
- net /IO/A_OUT_2_R: track 30.3 -> 107.0 mm
- net /input selector/A_OUT_3_L: track 0.00 -> 72.3 mm
- net +3.3V: track 0.00 -> 66.0 mm
- net /input selector/A_OUT_3_R: track 0.00 -> 55.8 mm
- net /input selector/A_OUT_L: track 12.5 -> 67.5 mm
- net /input selector/A_IN_R: track 22.9 -> 76.3 mm
- net /input selector/A_IN_L: track 25.0 -> 72.8 mm
- net /MCU/IO_SCL: track 4.12 -> 45.1 mm
- net /MCU/IO_SDA: track 4.12 -> 43.5 mm
- net /input selector/A_OUT_R: track 7.73 -> 40.1 mm
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Other:
- board size 374 x 202 mm -> 448 x 243 mm

Commit message: PCB layout updates, Power supply consolidation
Combined power supply boards. More PCB layout. PCB net assignment. Added mounting holes to boards. Front panel control / display layout. Various footprint updates / changes.
Parts:
- removed C1: 0.1uF, Capacitor_SMD:C_1812_4532Metric_Pad1.30x3.40mm_HandSolder
- removed F1: 500mA, preamp:01110501Z_3AG
- removed H13, H14, H15, H16, H5, H6, H7, H8: MountingHole, MountingHole:MountingHole_3.2mm_M3
- removed J1, J14, J5, J6: Screw_Terminal_01x03, TerminalBlock_Phoenix:TerminalBlock_Phoenix_MKDS-3-3-5.08_1x03_P5.08mm_Horizontal
- removed J11, J12, J13: Conn_01x02_Male, Connector_JST:JST_EH_B2B-EH-A_1x02_P2.50mm_Vertical
- removed J2: Conn_01x02_Female, Connector_JST:JST_EH_B2B-EH-A_1x02_P2.50mm_Vertical
- added F4: 500mA, preamp:01110501Z_3AG, F.Cu at (12.8, 151.5)
- C17, C18: moved to B.Cu
- J10, J9: value Conn_01x03_Male -> Conn_01x02_Male; footprint Connector_JST:JST_EH_B3B-EH-A_1x03_P2.50mm_Vertical -> Connector_PinHeader_2.54mm:PinHeader_1x02_P2.54mm_Vertical
- J17, J18: footprint Connector_PinHeader_2.54mm:PinHeader_1x02_P2.54mm_Vertical -> Connector_JST:JST_EH_B2B-EH-A_1x02_P2.50mm_Vertical
- J3: value Conn_01x02_Female -> Conn_01x04_Male; footprint Connector_JST:JST_EH_B2B-EH-A_1x02_P2.50mm_Vertical -> Connector_JST:JST_EH_B4B-EH-A_1x04_P2.50mm_Vertical
- J4: value Conn_01x02_Male -> Conn_01x02_Female; footprint Connector_PinHeader_2.54mm:PinHeader_1x02_P2.54mm_Vertical -> Connector_JST:JST_EH_B2B-EH-A_1x02_P2.50mm_Vertical
- J8: value Conn_01x03_Male -> Conn_01x04_Male; footprint Connector_JST:JST_EH_B3B-EH-A_1x03_P2.50mm_Vertical -> Connector_JST:JST_EH_B4B-EH-A_1x04_P2.50mm_Vertical
- moved H11 182.5 mm to (4.00, 165.0)
- moved H9 168.5 mm to (4.00, 86.0)
- moved J18 90.4 mm to (276.5, 60.9), turned to 180 degrees
- moved H12 89.0 mm to (102.0, 165.0)
- moved C17 86.0 mm to (270.5, 52.5), turned to 270 degrees
- moved C18 80.9 mm to (281.0, 25.8), turned to 270 degrees
- moved J15 78.9 mm to (230.5, 52.0)
- moved J16 78.9 mm to (230.5, 37.5)
- moved J19 78.9 mm to (301.8, 49.0)
- moved R11 78.9 mm to (257.2, 38.8)
- moved R12 78.9 mm to (257.2, 36.2)
- moved R13 78.9 mm to (270.2, 47.7)
- moved R14 78.9 mm to (270.2, 23.5)
- moved R15 78.9 mm to (270.2, 26.1)
- moved R16 78.9 mm to (270.2, 31.1)
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Connections:
- net /+-15V PWR SUPPLY/AC_N renamed /DC_PWR SUPPLY/AC_N
- F2 pad 2: /+-15V PWR SUPPLY/AC_HOT -> /DC_PWR SUPPLY/AC_HOT
- F3 pad 2: /+-15V PWR SUPPLY/AC_HOT -> /DC_PWR SUPPLY/AC_HOT
- J10 pad 1: +15V -> /DC_PWR SUPPLY/-15
- J10 pad 2: GND -> -15V
- J19 pad 3: /front panel/FP_INTA -> /MCU/ENC_INT
- J19 pad 4: /MCU/ENC_INT -> /front panel/FP_INTA
- J3 pad 1: /AC input/STBY_CTRL_1 -> +15V
- J3 pad 2: /AC input/STBY_CTRL_2 -> -15V
- J4 pad 1: /+-15V PWR SUPPLY/AC_HOT -> /DC_PWR SUPPLY/STBY_CTRL_1
- J4 pad 2: Net-(J4-Pad2) -> /DC_PWR SUPPLY/STBY_CTRL_2
- J7 pad 1: /+-15V PWR SUPPLY/AC_HOT -> /DC_PWR SUPPLY/AC_HOT
- J8 pad 2: GND -> -15V
- J8 pad 3: -15V -> GND
- J84 pad 3: /front panel/FP_INTA -> /MCU/ENC_INT
- J84 pad 4: /MCU/ENC_INT -> /front panel/FP_INTA
- J9 pad 1: +15V -> /DC_PWR SUPPLY/+15
- J9 pad 2: GND -> +15V
- PS1 pad 4: +15V -> /DC_PWR SUPPLY/+15
- PS2 pad 2: Net-(F2-Pad1) -> Net-(F3-Pad1)
- PS2 pad 3: -15V -> /DC_PWR SUPPLY/-15
- PS3 pad 2: Net-(F3-Pad1) -> Net-(F4-Pad1)
- U3 pad 12: /MCU/FP_SDA -> /MCU/SD3
- U3 pad 13: /MCU/FP_SCL -> /MCU/SC3
- U3 pad 15: /MCU/SD3 -> /Volume Control/DAC_SDA
- U3 pad 16: /MCU/SC3 -> /Volume Control/DAC_SCL
- U3 pad 8: /Volume Control/DAC_SDA -> /MCU/FP_SDA
- U3 pad 9: /Volume Control/DAC_SCL -> /MCU/FP_SCL
- U7 pad 11: /AC input/STBY_CTRL_1 -> /DC_PWR SUPPLY/STBY_CTRL_1
- U7 pad 12: /AC input/STBY_CTRL_2 -> /DC_PWR SUPPLY/STBY_CTRL_2
Routing:
- net +5V: track 1102.0 -> 400.3 mm, vias 1 -> 2
- net GND: track 617.1 -> 38.2 mm
- net /DC_PWR SUPPLY/AC_N: track 0.00 -> 114.7 mm
- net /front panel/FP_LED_DT: track 24.9 -> 102.9 mm
- net -15V: track 432.6 -> 490.6 mm
- net +15V: track 401.9 -> 457.6 mm
- net /front panel/FP_INTA: track 0.00 -> 38.1 mm
- net /MCU/ENC_INT: track 0.00 -> 38.1 mm
- net /DC_PWR SUPPLY/AC_HOT: track 0.00 -> 31.0 mm
- net Net-(F2-Pad1): track 0.00 -> 24.8 mm
- net /MCU/SCM: track 4.95 -> 29.7 mm
- net /MCU/SDM: track 4.95 -> 27.4 mm
- net /MCU/SC3: track 4.65 -> 27.0 mm
- net /MCU/FP_SDA: track 0.00 -> 19.9 mm
- net /MCU/SD3: track 4.11 -> 23.9 mm
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- added copper zone on F.Cu, net (none)
- removed copper zone on B.Cu, net (none)
Other:
- board size 448 x 243 mm -> 384.5 x 218 mm

Commit message: Power supply filter Implementation
Added pi filter on output of DC supplies. PCB layout update on the power supply board.
Parts:
- added C49: 470uF, Capacitor_THT:CP_Radial_D12.5mm_P5.00mm, F.Cu at (35.0, 156.0)
- added C50: 470uF, Capacitor_THT:CP_Radial_D12.5mm_P5.00mm, F.Cu at (35.0, 184.0)
- added C51: 470uF, Capacitor_THT:CP_Radial_D12.5mm_P5.00mm, F.Cu at (35.0, 212.0)
- added C52: 470uF, Capacitor_THT:CP_Radial_D12.5mm_P5.00mm, F.Cu at (35.0, 170.0)
- added C53: 470uF, Capacitor_THT:CP_Radial_D12.5mm_P5.00mm, F.Cu at (35.0, 198.0)
- added C54: 470uF, Capacitor_THT:CP_Radial_D12.5mm_P5.00mm, F.Cu at (35.0, 226.0)
- added K1: G6JU, preamp:Relay_DPDT_Omron_G6JU-2P-Y, F.Cu at (57.0, 177.5)
- added L1: 150uH, Inductor_THT:L_Axial_L23.4mm_D12.7mm_P7.62mm_Vertical_Vishay_IHA-203, F.Cu at (47.3, 162.2)
- added L2: 150uH, Inductor_THT:L_Axial_L23.4mm_D12.7mm_P7.62mm_Vertical_Vishay_IHA-203, F.Cu at (47.3, 190.4)
- added L3: 150uH, Inductor_THT:L_Axial_L23.4mm_D12.7mm_P7.62mm_Vertical_Vishay_IHA-203, F.Cu at (47.3, 218.5)
- moved C17 233.6 mm to (46.0, 117.0)
- moved C18 233.6 mm to (56.5, 90.3)
- moved H17 233.6 mm to (6.00, 86.0)
- moved H18 233.6 mm to (77.0, 86.0)
- moved H19 233.6 mm to (6.00, 124.0)
- moved H20 233.6 mm to (77.0, 124.0)
- moved J15 233.6 mm to (5.98, 116.5)
- moved J16 233.6 mm to (5.98, 102.0)
- moved J18 233.6 mm to (52.0, 125.4)
- moved J19 233.6 mm to (77.2, 113.5)
- moved J61 233.6 mm to (69.2, 84.2)
- moved R11 233.6 mm to (32.8, 103.3)
- moved R12 233.6 mm to (32.8, 100.7)
- moved R13 233.6 mm to (45.8, 112.2)
- moved R14 233.6 mm to (45.8, 88.0)
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Connections:
- PS1 pad 4: /DC_PWR SUPPLY/+15 -> Net-(C49-Pad1)
- PS2 pad 3: /DC_PWR SUPPLY/-15 -> Net-(C50-Pad1)
- PS3 pad 4: +5V -> Net-(C51-Pad1)
Routing:
- net /DC_PWR SUPPLY/+15: track 0.00 -> 54.2 mm
- net /DC_PWR SUPPLY/-15: track 0.00 -> 51.7 mm
- net Net-(C50-Pad1): track 0.00 -> 37.9 mm
- net Net-(C51-Pad1): track 0.00 -> 37.2 mm
- net Net-(C49-Pad1): track 0.00 -> 37.0 mm
- net -15V: track 490.6 -> 525.7 mm
- net +5V: track 400.3 -> 434.2 mm
- net /DC_PWR SUPPLY/AC_HOT: track 31.0 -> 61.6 mm
- net +15V: track 457.6 -> 484.7 mm
- net Net-(F4-Pad1): track 0.00 -> 21.3 mm
- net GND: track 38.2 -> 21.1 mm
- net /front panel/FP_LED_DT: track 102.9 -> 87.1 mm
- net /DC_PWR SUPPLY/STBY_CTRL_1: track 0.00 -> 13.0 mm
- net /DC_PWR SUPPLY/STBY_CTRL_2: track 0.00 -> 13.0 mm
- net /DC_PWR SUPPLY/AC_N: track 114.7 -> 104.1 mm
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Other:
- board size 384.5 x 218 mm -> 345 x 263 mm
