File: preamp-layout/preamp-kicad/_autosave-preamp.kicad_pcb (KiCad board)
At the start: 2 copper layers, 359.4 x 351.2 mm, 430 parts, among them J1 Screw_Terminal_01x03, J10 Conn_01x03_Male, J11 Conn_01x02_Male, J12 Conn_01x02_Male, J13 Conn_01x02_Male, J14 Screw_Terminal_01x03, J15 Conn_01x02_Male, J16 Conn_01x02_Male, J17 Conn_01x02_Female, J18 Conn_01x02_Female, J19 Conn_01x05_Female, J2 Conn_01x02_Female, J20 Conn_01x03_Male, J26 Conn_01x18_Male, J27 Conn_01x08_Male, J28 Conn_01x18_Female, J29 Conn_01x08_Female, J3 Conn_01x02_Female, J30 Conn_01x04_Female, J32 Conn_01x03_Male, J35 Conn_01x05_Male, J36 Conn_01x05_Female, J37 Conn_01x08_Male, J38 Conn_01x03_Male, J4 Conn_01x02_Male, J42 Conn_01x03_Female, J43 Conn_01x03_Female, J44 Conn_01x02_Female, J47 Conn_01x02_Male, J48 Conn_01x02_Male, J49 Conn_01x03_Female, J5 Screw_Terminal_01x03, J50 Conn_01x03_Male, J51 Conn_01x02_Male, J52 Conn_01x03_Male, J54 Conn_01x03_Male, J55 Conn_01x02_Male, J56 Conn_01x03_Male, J57 Conn_01x02_Male, J58 Conn_01x03_Male, J6 Screw_Terminal_01x03, J61 Conn_01x03_Male, J62 Conn_01x03_Male, J66 Conn_01x03_Male, J67 Conn_01x03_Male, J68 Conn_01x03_Female, J69 Conn_01x03_Male, J7 Screw_Terminal_01x03, J70 XLR3, J71 XLR3, J72 XLR3, J73 XLR3, J74 Conn_01x03_Female, J75 Conn_01x03_Female, J76 Conn_01x03_Female, J77 Conn_01x03_Female, J78 Conn_01x03_Female, J79 Conn_01x03_Female, J8 Conn_01x03_Male, J80 Conn_01x03_Female, J81 Conn_01x03_Female, J82 Conn_01x02_Male, J83 Conn_01x02_Male, J84 Conn_01x05_Female, J9 Conn_01x03_Male, J95 Conn_01x03_Male, J96 Conn_01x03_Male, K2 G6JU, K7 G6JU, K8 G6JU, T1 Transformer_1P_2S, T2 Transformer_1P_2S, U1 LM7815, U10 DG408DY, U11 DAC5574, U12 TL074CDR, U13 NJM2068M, U14 THAT2181, U15 THAT2181, U16 NJM2068M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

Commit message: Balanced in/out update
Created THAT1646, THAT1280 schematic symbols an implemented in the balanced IO daughter card. Various layout updates as well, this is WIP.
Routing:
- net /input selector/A_OUT_L: track 0.00 -> 42.7 mm, vias 0 -> 1
- net /input selector/A_OUT_R: track 0.00 -> 34.4 mm, vias 0 -> 1
- removed copper zone on B.Cu, net GND
Changed lines of the file:
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@@
     (thickness 1.6)
     (drawings 48)
-    (tracks 505)
+    (tracks 519)
     (zones 0)
     (modules 430)
@@
   (via (at 306.75 91.25) (size 0.8) (drill 0.4) (layers F.Cu B.Cu) (net 0))
   (via (at 303.25 87.75) (size 0.8) (drill 0.4) (layers F.Cu B.Cu) (net 0))
+  (via (at 134.2 67.4) (size 0.8) (drill 0.4) (layers F.Cu B.Cu) (net 30))
+  (via (at 134.2 64) (size 0.8) (drill 0.4) (layers F.Cu B.Cu) (net 28))
   (via (at 139.8 62.2) (size 0.8) (drill 0.4) (layers F.Cu B.Cu) (net 3))
   (via (at 140.2 45.4) (size 0.8) (drill 0.4) (layers F.Cu B.Cu) (net 3))
@@
   (segment (start 149.125 56.475) (end 149 56.6) (width 0.25) (layer B.Cu) (net 27))
   (segment (start 152.19 56.475) (end 149.125 56.475) (width 0.25) (layer B.Cu) (net 27))
+  (segment (start 131.9125 64) (end 131.8 63.8875) (width 0.25) (layer F.Cu) (net 28))
+  (segment (start 134.2 64) (end 131.9125 64) (width 0.25) (layer F.Cu) (net 28))
+  (segment (start 134.2 64) (end 136.2 66) (width 0.25) (layer B.Cu) (net 28))
+  (segment (start 136.2 66) (end 136.2 76.76359) (width 0.25) (layer B.Cu) (net 28))
+  (segment (start 136.2 76.76359) (end 137.5864 78.14999) (width 0.25) (layer B.Cu) (net 28))
+  (segment (start 137.5864 78.14999) (end 155.8 78.14999) (width 0.25) (layer B.Cu) (net 28))
+  (segment (start 155.8 78.14999) (end 162.25001 78.14999) (width 0.25) (layer B.Cu) (net 28))
   (segment (start 131.8 59.6) (end 127.8 55.6) (width 0.25) (layer F.Cu) (net 29))
   (segment (start 131.8 60.9125) (end 131.8 59.6) (width 0.25) (layer F.Cu) (net 29))
+  (segment (start 131.9125 67.4) (end 131.8 67.5125) (width 0.25) (layer F.Cu) (net 30))
+  (segment (start 134.2 67.4) (end 131.9125 67.4) (width 0.25) (layer F.Cu) (net 30))
+  (segment (start 134.2 67.4) (end 134.2 75.4) (width 0.25) (layer B.Cu) (net 30))
+  (segment (start 134.2 75.4) (end 137.4 78.6) (width 0.25) (layer B.Cu) (net 30))
+  (segment (start 137.4 78.6) (end 156.8 78.6) (width 0.25) (layer B.Cu) (net 30))
   (segment (start 179.9 71.845) (end 177.475 71.845) (width 0.25) (layer F.Cu) (net 31))
   (segment (start 188.535 70.2575) (end 187.5425 71.25) (width 0.25) (layer B.Cu) (net 31))
@@
   (segment (start 127.8 73) (end 128 73.2) (width 0.25) (layer F.Cu) (net 325))
   (segment (start 127.8 68.08) (end 127.8 71.8) (width 0.25) (layer F.Cu) (net 325))
-  (zone (net 3) (net_name GND) (layer B.Cu) (hatch edge 0.508)
-    (connect_pads (clearance 0.508))
-    (min_thickness 0.254)
-    (fill yes (arc_segments 32) (thermal_gap 0.508) (thermal_bridge_width 0.508))
-    (polygon
-      (pts
-        (xy 200.6 81.8) (xy 113.2 81.8) (xy 113.2 23.4) (xy 200.6 23.4)
-      )
-    )
-  )
 )
